File: design.kicad_pcb (KiCad board)
At the start: 2 copper layers, 25 x 22.9 mm, 14 parts, among them J1 Conn_01x02, J2 Conn_01x02, J3 Conn_01x03, J4 Conn_01x03, U1 TPS61099YFFT

Commit message: Update design.kicad_pcb
Parts:
- removed C1, C2, C3, C4: C_Small, Capacitor_SMD:C_0805_2012Metric
- removed J1, J2: Conn_01x02, Connector_PinHeader_2.54mm:PinHeader_1x02_P2.54mm_Vertical
- removed J3, J4: Conn_01x03, Connector_PinHeader_2.54mm:PinHeader_1x03_P2.54mm_Vertical
- removed JP1, JP2: SolderJumper_2_Open, Jumper:SolderJumper-2_P1.3mm_Open_RoundedPad1.0x1.5mm
- removed L1: L_Small, Inductor_SMD:L_1008_2520Metric
- removed R1, R2: R_Small, Resistor_SMD:R_0805_2012Metric
- removed U1: TPS61099YFFT, Converter_DCDC_custom:BGA6N40P3X2_122X88X62N
Routing:
- net En: track 19.9 -> 0.00 mm, vias 1 -> 0
- net Vin: track 14.5 -> 0.00 mm, vias 2 -> 0
- net FB: track 8.82 -> 0.00 mm
- net GND: track 3.05 -> 0.00 mm, vias 36 -> 0
- net Vout: track 2.80 -> 0.00 mm
- net SW: track 2.80 -> 0.00 mm
- removed copper zone on B.Cu, net GND
- removed copper zone on F.Cu, net GND
- removed copper zone on F.Cu, net SW
- removed copper zone on F.Cu, net Vin
- removed copper zone on F.Cu, net Vout
Other:
- board text removed: "EN"
- board text removed: "GND"
- board text removed: "Vin"
- board text removed: "Vout"

Commit message: Update design.kicad_pcb
Parts:
- added C1: 0-50pF, Capacitor_SMD:C_0805_2012Metric, F.Cu at (197.8, 99.8)
- added C10: 0-50pF, Capacitor_SMD:C_0805_2012Metric, F.Cu at (172.5, 122.6)
- added C11: 0-50pF, Capacitor_SMD:C_0805_2012Metric, F.Cu at (180.9, 113.0)
- added C12: 0-50pF, Capacitor_SMD:C_0805_2012Metric, F.Cu at (216.5, 79.9)
- added C13: 0-50pF, Capacitor_SMD:C_0805_2012Metric, F.Cu at (189.3, 109.4)
- added C16: 100nF, Capacitor_SMD:C_0805_2012Metric, F.Cu at (172.5, 125.6)
- added C17: 100nF, Capacitor_SMD:C_0805_2012Metric, F.Cu at (176.9, 119.6)
- added C18: 100nF, Capacitor_SMD:C_0805_2012Metric, F.Cu at (180.9, 116.0)
- added C19: 100nF, Capacitor_SMD:C_0805_2012Metric, F.Cu at (185.4, 113.0)
- added C2: 0-50pF, Capacitor_SMD:C_0805_2012Metric, F.Cu at (221.8, 73.3)
- added C3: 0-50pF, Capacitor_SMD:C_0805_2012Metric, F.Cu at (165.5, 132.8)
- added C4: 0-50pF, Capacitor_SMD:C_0805_2012Metric, F.Cu at (206.2, 91.2)
- added C5: 100nF, Capacitor_SMD:C_0805_2012Metric, F.Cu at (230.2, 66.7)
- added C6: 100nF, Capacitor_SMD:C_0805_2012Metric, F.Cu at (172.5, 119.6)
- added C7: 100nF, Capacitor_SMD:C_0805_2012Metric, F.Cu at (189.3, 106.4)
- added C8: 100nF, Capacitor_SMD:C_0805_2012Metric, F.Cu at (221.8, 76.3)
- added D10: WS2812B, LED_SMD:LED_WS2812B_PLCC4_5.0x5.0mm_P3.2mm, F.Cu at (132.4, 101.6)
- added D11: WS2812B, LED_SMD:LED_WS2812B_PLCC4_5.0x5.0mm_P3.2mm, F.Cu at (166.1, 114.8)
- added D12: WS2812B, LED_SMD:LED_WS2812B_PLCC4_5.0x5.0mm_P3.2mm, F.Cu at (136.9, 81.7)
- added D13: WS2812B, LED_SMD:LED_WS2812B_PLCC4_5.0x5.0mm_P3.2mm, F.Cu at (206.9, 68.5)
- added D14: WS2812B, LED_SMD:LED_WS2812B_PLCC4_5.0x5.0mm_P3.2mm, F.Cu at (115.5, 132.6)
- added D15: WS2812B, LED_SMD:LED_WS2812B_PLCC4_5.0x5.0mm_P3.2mm, F.Cu at (124.0, 112.7)
- added D16: WS2812B, LED_SMD:LED_WS2812B_PLCC4_5.0x5.0mm_P3.2mm, F.Cu at (206.9, 75.1)
- added D17: WS2812B, LED_SMD:LED_WS2812B_PLCC4_5.0x5.0mm_P3.2mm, F.Cu at (149.2, 128.0)
- added D18: WS2812B, LED_SMD:LED_WS2812B_PLCC4_5.0x5.0mm_P3.2mm, F.Cu at (124.0, 106.1)
- added D19: WS2812B, LED_SMD:LED_WS2812B_PLCC4_5.0x5.0mm_P3.2mm, F.Cu at (182.9, 108.2)
- added D20: WS2812B, LED_SMD:LED_WS2812B_PLCC4_5.0x5.0mm_P3.2mm, F.Cu at (166.1, 101.6)
- added D21: WS2812B, LED_SMD:LED_WS2812B_PLCC4_5.0x5.0mm_P3.2mm, F.Cu at (173.3, 68.5)
- added D22: WS2812B, LED_SMD:LED_WS2812B_PLCC4_5.0x5.0mm_P3.2mm, F.Cu at (164.8, 68.5)
- added D23: WS2812B, LED_SMD:LED_WS2812B_PLCC4_5.0x5.0mm_P3.2mm, F.Cu at (132.4, 88.3)
- added D24: WS2812B, LED_SMD:LED_WS2812B_PLCC4_5.0x5.0mm_P3.2mm, F.Cu at (115.5, 99.5)
- added D25: WS2812B, LED_SMD:LED_WS2812B_PLCC4_5.0x5.0mm_P3.2mm, F.Cu at (132.4, 121.4)
- added D26: WS2812B, LED_SMD:LED_WS2812B_PLCC4_5.0x5.0mm_P3.2mm, F.Cu at (149.2, 101.6)
- added D27: WS2812B, LED_SMD:LED_WS2812B_PLCC4_5.0x5.0mm_P3.2mm, F.Cu at (115.5, 119.4)
- added D28: WS2812B, LED_SMD:LED_WS2812B_PLCC4_5.0x5.0mm_P3.2mm, F.Cu at (139.6, 75.1)
- added D29: WS2812B, LED_SMD:LED_WS2812B_PLCC4_5.0x5.0mm_P3.2mm, F.Cu at (190.1, 68.5)
- added D3: WS2812B, LED_SMD:LED_WS2812B_PLCC4_5.0x5.0mm_P3.2mm, F.Cu at (115.5, 106.1)
- added D30: WS2812B, LED_SMD:LED_WS2812B_PLCC4_5.0x5.0mm_P3.2mm, F.Cu at (115.5, 112.7)
- added D31: WS2812B, LED_SMD:LED_WS2812B_PLCC4_5.0x5.0mm_P3.2mm, F.Cu at (140.8, 121.4)
- added D32: WS2812B, LED_SMD:LED_WS2812B_PLCC4_5.0x5.0mm_P3.2mm, F.Cu at (131.2, 75.1)
- added D33: WS2812B, LED_SMD:LED_WS2812B_PLCC4_5.0x5.0mm_P3.2mm, F.Cu at (174.5, 101.6)
- added D34: WS2812B, LED_SMD:LED_WS2812B_PLCC4_5.0x5.0mm_P3.2mm, F.Cu at (132.4, 114.8)
- added D35: WS2812B, LED_SMD:LED_WS2812B_PLCC4_5.0x5.0mm_P3.2mm, F.Cu at (199.7, 88.3)
- added D36: WS2812B, LED_SMD:LED_WS2812B_PLCC4_5.0x5.0mm_P3.2mm, F.Cu at (182.9, 88.3)
- added D37: WS2812B, LED_SMD:LED_WS2812B_PLCC4_5.0x5.0mm_P3.2mm, F.Cu at (157.6, 108.2)
- added D38: WS2812B, LED_SMD:LED_WS2812B_PLCC4_5.0x5.0mm_P3.2mm, F.Cu at (157.6, 121.4)
- added D39: WS2812B, LED_SMD:LED_WS2812B_PLCC4_5.0x5.0mm_P3.2mm, F.Cu at (179.0, 81.7)
- added D4: WS2812B, LED_SMD:LED_WS2812B_PLCC4_5.0x5.0mm_P3.2mm, F.Cu at (157.6, 114.8)
- added D40: WS2812B, LED_SMD:LED_WS2812B_PLCC4_5.0x5.0mm_P3.2mm, F.Cu at (166.1, 121.4)
- added D41: WS2812B, LED_SMD:LED_WS2812B_PLCC4_5.0x5.0mm_P3.2mm, F.Cu at (132.4, 108.2)
- added D42: WS2812B, LED_SMD:LED_WS2812B_PLCC4_5.0x5.0mm_P3.2mm, F.Cu at (149.2, 114.8)
- added D43: WS2812B, LED_SMD:LED_WS2812B_PLCC4_5.0x5.0mm_P3.2mm, F.Cu at (145.3, 81.7)
- added D44: WS2812B, LED_SMD:LED_WS2812B_PLCC4_5.0x5.0mm_P3.2mm, F.Cu at (204.2, 81.7)
- added D45: WS2812B, LED_SMD:LED_WS2812B_PLCC4_5.0x5.0mm_P3.2mm, F.Cu at (181.7, 75.1)
- added D46: WS2812B, LED_SMD:LED_WS2812B_PLCC4_5.0x5.0mm_P3.2mm, F.Cu at (166.1, 108.2)
- added D47: WS2812B, LED_SMD:LED_WS2812B_PLCC4_5.0x5.0mm_P3.2mm, F.Cu at (215.4, 68.5)
- added D48: WS2812B, LED_SMD:LED_WS2812B_PLCC4_5.0x5.0mm_P3.2mm, F.Cu at (148.0, 75.1)
- added D49: WS2812B, LED_SMD:LED_WS2812B_PLCC4_5.0x5.0mm_P3.2mm, F.Cu at (139.6, 68.5)
- added D5: WS2812B, LED_SMD:LED_WS2812B_PLCC4_5.0x5.0mm_P3.2mm, F.Cu at (124.0, 132.6)
- added D50: WS2812B, LED_SMD:LED_WS2812B_PLCC4_5.0x5.0mm_P3.2mm, F.Cu at (140.8, 108.2)
- added D51: WS2812B, LED_SMD:LED_WS2812B_PLCC4_5.0x5.0mm_P3.2mm, F.Cu at (156.4, 68.5)
- added D52: WS2812B, LED_SMD:LED_WS2812B_PLCC4_5.0x5.0mm_P3.2mm, F.Cu at (187.4, 81.7)
- added D53: WS2812B, LED_SMD:LED_WS2812B_PLCC4_5.0x5.0mm_P3.2mm, F.Cu at (131.2, 68.5)
- added D54: WS2812B, LED_SMD:LED_WS2812B_PLCC4_5.0x5.0mm_P3.2mm, F.Cu at (166.1, 88.3)
- added D55: WS2812B, LED_SMD:LED_WS2812B_PLCC4_5.0x5.0mm_P3.2mm, F.Cu at (140.8, 94.9)
- added D56: WS2812B, LED_SMD:LED_WS2812B_PLCC4_5.0x5.0mm_P3.2mm, F.Cu at (124.0, 99.5)
- added D57: WS2812B, LED_SMD:LED_WS2812B_PLCC4_5.0x5.0mm_P3.2mm, F.Cu at (149.2, 94.9)
- added D58: WS2812B, LED_SMD:LED_WS2812B_PLCC4_5.0x5.0mm_P3.2mm, F.Cu at (215.4, 75.1)
- added D59: WS2812B, LED_SMD:LED_WS2812B_PLCC4_5.0x5.0mm_P3.2mm, F.Cu at (132.4, 94.9)
- added D6: WS2812B, LED_SMD:LED_WS2812B_PLCC4_5.0x5.0mm_P3.2mm, F.Cu at (190.1, 75.1)
- added D60: WS2812B, LED_SMD:LED_WS2812B_PLCC4_5.0x5.0mm_P3.2mm, F.Cu at (157.6, 128.0)
- added D61: WS2812B, LED_SMD:LED_WS2812B_PLCC4_5.0x5.0mm_P3.2mm, F.Cu at (198.5, 75.1)
- added D62: WS2812B, LED_SMD:LED_WS2812B_PLCC4_5.0x5.0mm_P3.2mm, F.Cu at (128.4, 81.7)
- added D63: WS2812B, LED_SMD:LED_WS2812B_PLCC4_5.0x5.0mm_P3.2mm, F.Cu at (174.5, 88.3)
- added D64: WS2812B, LED_SMD:LED_WS2812B_PLCC4_5.0x5.0mm_P3.2mm, F.Cu at (140.8, 101.6)
- added D65: WS2812B, LED_SMD:LED_WS2812B_PLCC4_5.0x5.0mm_P3.2mm, F.Cu at (148.0, 68.5)
- added D66: WS2812B, LED_SMD:LED_WS2812B_PLCC4_5.0x5.0mm_P3.2mm, F.Cu at (182.9, 94.9)
- added D67: WS2812B, LED_SMD:LED_WS2812B_PLCC4_5.0x5.0mm_P3.2mm, F.Cu at (140.8, 128.0)
- added D68: WS2812B, LED_SMD:LED_WS2812B_PLCC4_5.0x5.0mm_P3.2mm, F.Cu at (157.6, 88.3)
- added D69: WS2812B, LED_SMD:LED_WS2812B_PLCC4_5.0x5.0mm_P3.2mm, F.Cu at (162.1, 81.7)
- added D7: WS2812B, LED_SMD:LED_WS2812B_PLCC4_5.0x5.0mm_P3.2mm, F.Cu at (115.5, 126.0)
- added D70: WS2812B, LED_SMD:LED_WS2812B_PLCC4_5.0x5.0mm_P3.2mm, F.Cu at (157.6, 94.9)
- added D71: WS2812B, LED_SMD:LED_WS2812B_PLCC4_5.0x5.0mm_P3.2mm, F.Cu at (195.8, 81.7)
- added D72: WS2812B, LED_SMD:LED_WS2812B_PLCC4_5.0x5.0mm_P3.2mm, F.Cu at (153.7, 81.7)
- added D73: WS2812B, LED_SMD:LED_WS2812B_PLCC4_5.0x5.0mm_P3.2mm, F.Cu at (140.8, 114.8)
- added D74: WS2812B, LED_SMD:LED_WS2812B_PLCC4_5.0x5.0mm_P3.2mm, F.Cu at (124.0, 119.4)
- added D75: WS2812B, LED_SMD:LED_WS2812B_PLCC4_5.0x5.0mm_P3.2mm, F.Cu at (199.7, 94.9)
- added D76: WS2812B, LED_SMD:LED_WS2812B_PLCC4_5.0x5.0mm_P3.2mm, F.Cu at (191.3, 94.9)
- added D77: WS2812B, LED_SMD:LED_WS2812B_PLCC4_5.0x5.0mm_P3.2mm, F.Cu at (174.5, 114.8)
- added D78: WS2812B, LED_SMD:LED_WS2812B_PLCC4_5.0x5.0mm_P3.2mm, F.Cu at (164.8, 75.1)
- added D79: WS2812B, LED_SMD:LED_WS2812B_PLCC4_5.0x5.0mm_P3.2mm, F.Cu at (174.5, 94.9)
- added D8: WS2812B, LED_SMD:LED_WS2812B_PLCC4_5.0x5.0mm_P3.2mm, F.Cu at (149.2, 108.2)
- added D80: WS2812B, LED_SMD:LED_WS2812B_PLCC4_5.0x5.0mm_P3.2mm, F.Cu at (223.8, 68.5)
- added D81: WS2812B, LED_SMD:LED_WS2812B_PLCC4_5.0x5.0mm_P3.2mm, F.Cu at (198.5, 68.5)
- added D82: WS2812B, LED_SMD:LED_WS2812B_PLCC4_5.0x5.0mm_P3.2mm, F.Cu at (157.6, 101.6)
- added D83: WS2812B, LED_SMD:LED_WS2812B_PLCC4_5.0x5.0mm_P3.2mm, F.Cu at (140.8, 88.3)
- added D84: WS2812B, LED_SMD:LED_WS2812B_PLCC4_5.0x5.0mm_P3.2mm, F.Cu at (173.3, 75.1)
- added D85: WS2812B, LED_SMD:LED_WS2812B_PLCC4_5.0x5.0mm_P3.2mm, F.Cu at (156.4, 75.1)
- added D86: WS2812B, LED_SMD:LED_WS2812B_PLCC4_5.0x5.0mm_P3.2mm, F.Cu at (170.5, 81.7)
- added D87: WS2812B, LED_SMD:LED_WS2812B_PLCC4_5.0x5.0mm_P3.2mm, F.Cu at (124.0, 126.0)
- added D88: WS2812B, LED_SMD:LED_WS2812B_PLCC4_5.0x5.0mm_P3.2mm, F.Cu at (115.5, 92.9)
- added D89: WS2812B, LED_SMD:LED_WS2812B_PLCC4_5.0x5.0mm_P3.2mm, F.Cu at (149.2, 88.3)
- added D9: WS2812B, LED_SMD:LED_WS2812B_PLCC4_5.0x5.0mm_P3.2mm, F.Cu at (149.2, 121.4)
- added D90: WS2812B, LED_SMD:LED_WS2812B_PLCC4_5.0x5.0mm_P3.2mm, F.Cu at (132.4, 128.0)
- added D91: WS2812B, LED_SMD:LED_WS2812B_PLCC4_5.0x5.0mm_P3.2mm, F.Cu at (191.3, 101.6)
- added D92: WS2812B, LED_SMD:LED_WS2812B_PLCC4_5.0x5.0mm_P3.2mm, F.Cu at (166.1, 128.0)
- added D93: WS2812B, LED_SMD:LED_WS2812B_PLCC4_5.0x5.0mm_P3.2mm, F.Cu at (174.5, 108.2)
- added D94: WS2812B, LED_SMD:LED_WS2812B_PLCC4_5.0x5.0mm_P3.2mm, F.Cu at (191.3, 88.3)
- added D95: WS2812B, LED_SMD:LED_WS2812B_PLCC4_5.0x5.0mm_P3.2mm, F.Cu at (166.1, 94.9)
- added D96: WS2812B, LED_SMD:LED_WS2812B_PLCC4_5.0x5.0mm_P3.2mm, F.Cu at (182.9, 101.6)
- added D97: WS2812B, LED_SMD:LED_WS2812B_PLCC4_5.0x5.0mm_P3.2mm, F.Cu at (124.0, 92.9)
- added D98: WS2812B, LED_SMD:LED_WS2812B_PLCC4_5.0x5.0mm_P3.2mm, F.Cu at (181.7, 68.5)
- added J1: TYPE-C-31-M-12, Snapeda:TYPE-C-31-M-12_HRO_TYPE-C-31-M-12, F.Cu at (117.4, 71.8)
- added JP1: TOG, Jumper:SolderJumper-2_P1.3mm_Open_RoundedPad1.0x1.5mm, F.Cu at (216.4, 86.1)
- added JP10: TOG, Jumper:SolderJumper-2_P1.3mm_Open_RoundedPad1.0x1.5mm, F.Cu at (220.9, 83.2)
- added JP11: AHLB, Jumper:SolderJumper-2_P1.3mm_Open_RoundedPad1.0x1.5mm, F.Cu at (210.6, 91.4)
- added JP12: TOG, Jumper:SolderJumper-2_P1.3mm_Open_RoundedPad1.0x1.5mm, F.Cu at (210.5, 95.0)
- added JP13: AHLB, Jumper:SolderJumper-2_P1.3mm_Open_RoundedPad1.0x1.5mm, F.Cu at (226.2, 76.5)
- added JP14: TOG, Jumper:SolderJumper-2_P1.3mm_Open_RoundedPad1.0x1.5mm, F.Cu at (169.9, 133.1)
- added JP15: AHLB, Jumper:SolderJumper-2_P1.3mm_Open_RoundedPad1.0x1.5mm, F.Cu at (181.3, 119.3)
- added JP16: TOG, Jumper:SolderJumper-2_P1.3mm_Open_RoundedPad1.0x1.5mm, F.Cu at (189.8, 112.7)
- added JP17: AHLB, Jumper:SolderJumper-2_P1.3mm_Open_RoundedPad1.0x1.5mm, F.Cu at (176.9, 125.8)
- added JP2: AHLB, Jumper:SolderJumper-2_P1.3mm_Open_RoundedPad1.0x1.5mm, F.Cu at (181.3, 122.8)
- added JP3: TOG, Jumper:SolderJumper-2_P1.3mm_Open_RoundedPad1.0x1.5mm, F.Cu at (202.1, 103.6)
- added JP4: AHLB, Jumper:SolderJumper-2_P1.3mm_Open_RoundedPad1.0x1.5mm, F.Cu at (202.2, 100.0)
- added JP5: TOG, Jumper:SolderJumper-2_P1.3mm_Open_RoundedPad1.0x1.5mm, F.Cu at (230.6, 72.9)
- added JP6: AHLB, Jumper:SolderJumper-2_P1.3mm_Open_RoundedPad1.0x1.5mm, F.Cu at (185.7, 116.3)
- added JP7: TOG, Jumper:SolderJumper-2_P1.3mm_Open_RoundedPad1.0x1.5mm, F.Cu at (197.7, 103.0)
- added JP8: AHLB, Jumper:SolderJumper-2_P1.3mm_Open_RoundedPad1.0x1.5mm, F.Cu at (193.7, 106.6)
- added R1: 5.1k, Resistor_SMD:R_0805_2012Metric, F.Cu at (172.5, 128.6)
- added R10: 1k, Resistor_SMD:R_0805_2012Metric, F.Cu at (212.0, 84.5)
- added R2: 5.1k, Resistor_SMD:R_0805_2012Metric, F.Cu at (206.2, 94.1)
- added R3: 2.4k, Resistor_SMD:R_0805_2012Metric, F.Cu at (212.0, 87.5)
- added R4: 13.3k, Resistor_SMD:R_0805_2012Metric, F.Cu at (221.8, 79.3)
- added R5: 1k, Resistor_SMD:R_0805_2012Metric, F.Cu at (230.2, 69.6)
- added R6: 1k, Resistor_SMD:R_0805_2012Metric, F.Cu at (226.2, 73.2)
- added R7: 1k, Resistor_SMD:R_0805_2012Metric, F.Cu at (234.6, 66.6)
- added R8: 1k, Resistor_SMD:R_0805_2012Metric, F.Cu at (216.5, 82.9)
- added R9: 1k, Resistor_SMD:R_0805_2012Metric, F.Cu at (176.9, 122.6)
- added U1: TTP223, Package_TO_SOT_SMD:SOT-23-6_Handsoldering, F.Cu at (160.3, 133.7)
- added U10: ATtiny1616-S, Package_SO:SOIC-20W_7.5x12.8mm_P1.27mm, F.Cu at (117.8, 82.4)
- added U2: TTP223, Package_TO_SOT_SMD:SOT-23-6_Handsoldering, F.Cu at (154.5, 133.7)
- added U3: TTP223, Package_TO_SOT_SMD:SOT-23-6_Handsoldering, F.Cu at (148.6, 133.7)
- added U4: TTP223, Package_TO_SOT_SMD:SOT-23-6_Handsoldering, F.Cu at (142.8, 133.7)
- added U6: TTP223, Package_TO_SOT_SMD:SOT-23-6_Handsoldering, F.Cu at (211.4, 80.7)
- added U7: TTP223, Package_TO_SOT_SMD:SOT-23-6_Handsoldering, F.Cu at (206.9, 87.3)
- added U8: TTP223, Package_TO_SOT_SMD:SOT-23-6_Handsoldering, F.Cu at (136.9, 133.7)
- added U9: TTP223, Package_TO_SOT_SMD:SOT-23-6_Handsoldering, F.Cu at (131.1, 133.7)
Other:
- board size 25 x 22.9 mm -> 149 x 107.8 mm

Commit message: update
Parts:
- removed U9: TTP223, Package_TO_SOT_SMD:SOT-23-6_Handsoldering
- added C14: 100nF, Capacitor_SMD:C_0805_2012Metric, F.Cu at (52.2, 68.6)
- added C15: 100nF, Capacitor_SMD:C_0805_2012Metric, F.Cu at (56.7, 68.6)
- added C20: 2.2uF, Capacitor_SMD:C_0805_2012Metric, F.Cu at (33.3, 89.3)
- added C21: 0.1uF, Capacitor_SMD:C_0805_2012Metric, F.Cu at (39.5, 109.1)
- added C22: 10uF, Capacitor_SMD:C_0805_2012Metric, F.Cu at (69.0, 114.7)
- added C23: 22uF, Capacitor_SMD:C_0805_2012Metric, F.Cu at (43.8, 79.7)
- added C24: 2.2uF, Capacitor_SMD:C_0805_2012Metric, F.Cu at (37.8, 84.8)
- added C25: 2.2uF, Capacitor_SMD:C_0805_2012Metric, F.Cu at (19.4, 130.4)
- added C26: 0.1uF, Capacitor_SMD:C_0805_2012Metric, F.Cu at (52.2, 71.6)
- added C27: 10uF, Capacitor_SMD:C_0805_2012Metric, F.Cu at (36.2, 116.3)
- added C9: 0-50pF, Capacitor_SMD:C_0805_2012Metric, F.Cu at (77.8, 94.8)
- added D1: WS2812B, LED_SMD:LED_WS2812B_PLCC4_5.0x5.0mm_P3.2mm, F.Cu at (130.4, 55.8)
- added D100: STAT, LED_SMD:LED_0603_1608Metric, F.Cu at (52.5, 78.0)
- added D101: Red, LED_SMD:LED_0603_1608Metric, F.Cu at (26.0, 105.7)
- added D102: Green, LED_SMD:LED_0603_1608Metric, F.Cu at (70.2, 121.6)
- added D2: WS2812B, LED_SMD:LED_WS2812B_PLCC4_5.0x5.0mm_P3.2mm, F.Cu at (139.4, 55.8)
- added D99: INOKB, LED_SMD:LED_0603_1608Metric, F.Cu at (40.8, 118.2)
- added JP9: TOG, Jumper:SolderJumper-2_P1.3mm_Open_RoundedPad1.0x1.5mm, F.Cu at (33.7, 96.1)
- added L1: 0.47uH, Inductor_SMD:L_0805_2012Metric, F.Cu at (73.2, 94.7)
- added TP10: BAT-, TestPoint:TestPoint_Pad_4.0x4.0mm, F.Cu at (40.3, 104.6)
- added TP9: BAT+, TestPoint:TestPoint_Pad_4.0x4.0mm, F.Cu at (56.2, 119.0)
- added U5: TTP223, Package_TO_SOT_SMD:SOT-23-6, F.Cu at (20.1, 95.8)
- C13: value 0-50pF -> 100nF
- C17, C18, C19: value 100nF -> 10uF
- D97: value WS2812B -> 5V; footprint LED_SMD:LED_WS2812B_PLCC4_5.0x5.0mm_P3.2mm -> LED_SMD:LED_0603_1608Metric
- D98: value WS2812B -> VBUS; footprint LED_SMD:LED_WS2812B_PLCC4_5.0x5.0mm_P3.2mm -> LED_SMD:LED_0603_1608Metric
- JP10, JP12, JP14, JP16: value TOG -> AHLB
- JP11, JP13, JP15: value AHLB -> TOG
- JP17: value AHLB -> ENBST; footprint Jumper:SolderJumper-2_P1.3mm_Open_RoundedPad1.0x1.5mm -> LED_SMD:LED_0603_1608Metric
- R1, R2: value 5.1k -> 1k
- R3: value 2.4k -> 1k
- R4: value 13.3k -> 5.1k
- R6: value 1k -> 5.1k
- R7: value 1k -> 2.4k
- R8: value 1k -> 13.3k
- U1, U2, U3, U4, U6, U7, U8: footprint Package_TO_SOT_SMD:SOT-23-6_Handsoldering -> Package_TO_SOT_SMD:SOT-23-6
- moved C5 210.1 mm to (27.8, 122.9)
- moved R5 205.2 mm to (32.2, 123.7)
- moved R6 198.2 mm to (29.4, 95.8)
- moved JP5 193.4 mm to (38.1, 91.1)
- moved R7 193.0 mm to (42.3, 82.6)
- moved JP11 189.3 mm to (21.8, 105.8)
- moved R3 188.2 mm to (27.8, 125.9)
- moved C4 187.1 mm to (22.6, 127.3)
- moved C8 185.8 mm to (39.5, 112.1)
- moved JP12 184.4 mm to (26.2, 102.6)
- moved JP13 184.2 mm to (42.2, 85.9)
- moved U6 183.6 mm to (31.4, 117.0)
- moved R10 183.4 mm to (32.2, 120.7)
- moved JP1 182.9 mm to (36.6, 119.6)
- moved R8 178.8 mm to (37.8, 87.8)
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Connections:
- C1 pad 1: touch_point_3 -> touch_point_1
- C10 pad 1: touch_point_7 -> touch_point_6
- C11 pad 1: touch_point_8 -> touch_point_7
- C12 pad 1: touch_point_5 -> touch_point_8
- C13 pad 1: touch_point_6 -> VCC
- C17 pad 1: VCC -> PGND
- C17 pad 2: PGND -> Net-(C17-Pad2)
- C18 pad 1: VCC -> PGND
- C18 pad 2: PGND -> +5V
- C19 pad 1: VCC -> PGND
- C19 pad 2: PGND -> +5V
- C2 pad 1: touch_point_4 -> touch_point_2
- C3 pad 1: touch_point_1 -> touch_point_3
- C4 pad 1: touch_point_2 -> touch_point_4
- D10 pad 2: Net-(D10-Pad2) -> Net-(D2-Pad4)
- D10 pad 4: 7out -> in
- D11 pad 2: Net-(D11-Pad2) -> Net-(D2-Pad4)
- D11 pad 4: Net-(D11-Pad4) -> in
- D12 pad 2: Net-(D12-Pad2) -> Net-(D2-Pad4)
- D12 pad 4: Net-(D12-Pad4) -> in
- D13 pad 2: Net-(D13-Pad2) -> Net-(D2-Pad4)
- D13 pad 4: Net-(D13-Pad4) -> in
- D14 pad 2: Net-(D14-Pad2) -> Net-(D2-Pad4)
- D14 pad 4: Net-(D14-Pad4) -> in
- D15 pad 2: Net-(D15-Pad2) -> Net-(D2-Pad4)
- D15 pad 4: Net-(D15-Pad4) -> in
- D16 pad 2: Net-(D16-Pad2) -> Net-(D2-Pad4)
- D16 pad 4: Net-(D16-Pad4) -> in
- D17 pad 2: Net-(D17-Pad2) -> Net-(D2-Pad4)
- D17 pad 4: Net-(D17-Pad4) -> in
- D18 pad 2: Net-(D18-Pad2) -> Net-(D2-Pad4)
- D18 pad 4: Net-(D10-Pad2) -> in
- D19 pad 2: Net-(D19-Pad2) -> Net-(D2-Pad4)
- D19 pad 4: Net-(D11-Pad2) -> in
- D20 pad 2: Net-(D20-Pad2) -> Net-(D2-Pad4)
- D20 pad 4: Net-(D12-Pad2) -> in
- D21 pad 2: Net-(D21-Pad2) -> Net-(D2-Pad4)
- D21 pad 4: Net-(D13-Pad2) -> in
- D22 pad 2: Net-(D22-Pad2) -> Net-(D2-Pad4)
- D22 pad 4: Net-(D14-Pad2) -> in
- D23 pad 2: Net-(D23-Pad2) -> Net-(D2-Pad4)
- D23 pad 4: Net-(D15-Pad2) -> in
- D24 pad 2: Net-(D24-Pad2) -> Net-(D2-Pad4)
- D24 pad 4: Net-(D16-Pad2) -> in
- D25 pad 2: Net-(D25-Pad2) -> Net-(D2-Pad4)
- D25 pad 4: Net-(D17-Pad2) -> in
- D26 pad 2: Net-(D26-Pad2) -> Net-(D2-Pad4)
- D26 pad 4: Net-(D18-Pad2) -> in
- D27 pad 2: Net-(D27-Pad2) -> Net-(D2-Pad4)
- D27 pad 4: Net-(D19-Pad2) -> in
- D28 pad 2: Net-(D28-Pad2) -> Net-(D2-Pad4)
- D28 pad 4: Net-(D20-Pad2) -> in
- D29 pad 2: Net-(D29-Pad2) -> Net-(D2-Pad4)
- D29 pad 4: Net-(D21-Pad2) -> in
- D3 pad 2: Net-(D11-Pad4) -> Net-(D2-Pad4)
- D30 pad 2: Net-(D30-Pad2) -> Net-(D2-Pad4)
- D30 pad 4: Net-(D22-Pad2) -> in
- D31 pad 2: Net-(D31-Pad2) -> Net-(D2-Pad4)
- D31 pad 4: Net-(D23-Pad2) -> in
- D32 pad 2: Net-(D32-Pad2) -> Net-(D2-Pad4)
- D32 pad 4: Net-(D24-Pad2) -> in
- D33 pad 2: Net-(D33-Pad2) -> Net-(D2-Pad4)
- D33 pad 4: Net-(D25-Pad2) -> in
- D34 pad 2: Net-(D34-Pad2) -> Net-(D2-Pad4)
- D34 pad 4: Net-(D26-Pad2) -> in
- D35 pad 2: Net-(D35-Pad2) -> Net-(D2-Pad4)
- D35 pad 4: Net-(D27-Pad2) -> in
- D36 pad 2: Net-(D36-Pad2) -> Net-(D2-Pad4)
- D36 pad 4: Net-(D28-Pad2) -> in
- D37 pad 2: Net-(D37-Pad2) -> Net-(D2-Pad4)
- D37 pad 4: Net-(D29-Pad2) -> in
- D38 pad 2: Net-(D38-Pad2) -> Net-(D2-Pad4)
- D38 pad 4: Net-(D30-Pad2) -> in
- D39 pad 2: Net-(D39-Pad2) -> Net-(D2-Pad4)
- D39 pad 4: Net-(D31-Pad2) -> in
- D4 pad 2: Net-(D12-Pad4) -> Net-(D2-Pad4)
- D4 pad 4: 1out -> in
- D40 pad 2: Net-(D40-Pad2) -> Net-(D2-Pad4)
- D40 pad 4: Net-(D32-Pad2) -> in
- D41 pad 2: Net-(D41-Pad2) -> Net-(D2-Pad4)
- D41 pad 4: Net-(D33-Pad2) -> in
- D42 pad 2: Net-(D42-Pad2) -> Net-(D2-Pad4)
- D42 pad 4: Net-(D34-Pad2) -> in
- D43 pad 2: Net-(D43-Pad2) -> Net-(D2-Pad4)
- D43 pad 4: Net-(D35-Pad2) -> in
- D44 pad 2: Net-(D44-Pad2) -> Net-(D2-Pad4)
- D44 pad 4: Net-(D36-Pad2) -> in
- D45 pad 2: Net-(D45-Pad2) -> Net-(D2-Pad4)
- D45 pad 4: Net-(D37-Pad2) -> in
- D46 pad 2: Net-(D46-Pad2) -> Net-(D2-Pad4)
- D46 pad 4: Net-(D38-Pad2) -> in
- D47 pad 2: Net-(D47-Pad2) -> Net-(D2-Pad4)
- D47 pad 4: Net-(D39-Pad2) -> in
- D48 pad 2: Net-(D48-Pad2) -> Net-(D2-Pad4)
- D48 pad 4: Net-(D40-Pad2) -> in
- D49 pad 2: Net-(D49-Pad2) -> Net-(D2-Pad4)
- D49 pad 4: Net-(D41-Pad2) -> in
- D5 pad 2: Net-(D13-Pad4) -> Net-(D2-Pad4)
- D5 pad 4: 2out -> in
- D50 pad 2: Net-(D50-Pad2) -> Net-(D2-Pad4)
- D50 pad 4: Net-(D42-Pad2) -> in
- D51 pad 2: Net-(D51-Pad2) -> Net-(D2-Pad4)
- D51 pad 4: Net-(D43-Pad2) -> in
- D52 pad 2: Net-(D52-Pad2) -> Net-(D2-Pad4)
- D52 pad 4: Net-(D44-Pad2) -> in
- D53 pad 2: Net-(D53-Pad2) -> Net-(D2-Pad4)
- D53 pad 4: Net-(D45-Pad2) -> in
- D54 pad 2: Net-(D54-Pad2) -> Net-(D2-Pad4)
- D54 pad 4: Net-(D46-Pad2) -> in
- D55 pad 2: Net-(D55-Pad2) -> Net-(D2-Pad4)
- D55 pad 4: Net-(D47-Pad2) -> in
- D56 pad 2: Net-(D56-Pad2) -> Net-(D2-Pad4)
- D56 pad 4: Net-(D48-Pad2) -> in
- D57 pad 2: Net-(D57-Pad2) -> Net-(D2-Pad4)
- D57 pad 4: Net-(D49-Pad2) -> in
- D58 pad 2: Net-(D58-Pad2) -> Net-(D2-Pad4)
- D58 pad 4: Net-(D50-Pad2) -> in
- D59 pad 2: Net-(D59-Pad2) -> Net-(D2-Pad4)
- D59 pad 4: Net-(D51-Pad2) -> in
- D6 pad 2: Net-(D14-Pad4) -> Net-(D2-Pad4)
- D6 pad 4: 3out -> in
- D60 pad 2: Net-(D60-Pad2) -> Net-(D2-Pad4)
- D60 pad 4: Net-(D52-Pad2) -> in
- D61 pad 2: Net-(D61-Pad2) -> Net-(D2-Pad4)
- D61 pad 4: Net-(D53-Pad2) -> in
- D62 pad 2: Net-(D62-Pad2) -> Net-(D2-Pad4)
- D62 pad 4: Net-(D54-Pad2) -> in
- D63 pad 2: Net-(D63-Pad2) -> Net-(D2-Pad4)
- D63 pad 4: Net-(D55-Pad2) -> in
- D64 pad 2: Net-(D64-Pad2) -> Net-(D2-Pad4)
- D64 pad 4: Net-(D56-Pad2) -> in
- D65 pad 2: Net-(D65-Pad2) -> Net-(D2-Pad4)
- D65 pad 4: Net-(D57-Pad2) -> in
- D66 pad 2: Net-(D66-Pad2) -> Net-(D2-Pad4)
- D66 pad 4: Net-(D58-Pad2) -> in
- D67 pad 2: Net-(D67-Pad2) -> Net-(D2-Pad4)
- D67 pad 4: Net-(D59-Pad2) -> in
- D68 pad 2: Net-(D68-Pad2) -> Net-(D2-Pad4)
- D68 pad 4: Net-(D60-Pad2) -> in
- D69 pad 2: Net-(D69-Pad2) -> Net-(D2-Pad4)
- D69 pad 4: Net-(D61-Pad2) -> in
- D7 pad 2: Net-(D15-Pad4) -> Net-(D2-Pad4)
- D7 pad 4: 4out -> in
- D70 pad 2: Net-(D70-Pad2) -> Net-(D2-Pad4)
- D70 pad 4: Net-(D62-Pad2) -> in
- D71 pad 2: Net-(D71-Pad2) -> Net-(D2-Pad4)
- D71 pad 4: Net-(D63-Pad2) -> in
- D72 pad 2: Net-(D72-Pad2) -> Net-(D2-Pad4)
- D72 pad 4: Net-(D64-Pad2) -> in
- D73 pad 2: Net-(D73-Pad2) -> Net-(D2-Pad4)
- D73 pad 4: Net-(D65-Pad2) -> in
- D74 pad 2: Net-(D74-Pad2) -> Net-(D2-Pad4)
- D74 pad 4: Net-(D66-Pad2) -> in
- D75 pad 2: Net-(D75-Pad2) -> Net-(D2-Pad4)
- D75 pad 4: Net-(D67-Pad2) -> in
- D76 pad 2: Net-(D76-Pad2) -> Net-(D2-Pad4)
- D76 pad 4: Net-(D68-Pad2) -> in
- D77 pad 2: Net-(D77-Pad2) -> Net-(D2-Pad4)
- D77 pad 4: Net-(D69-Pad2) -> in
- D78 pad 2: Net-(D78-Pad2) -> Net-(D2-Pad4)
- D78 pad 4: Net-(D70-Pad2) -> in
- D79 pad 2: Net-(D79-Pad2) -> Net-(D2-Pad4)
- D79 pad 4: Net-(D71-Pad2) -> in
- D8 pad 2: Net-(D16-Pad4) -> Net-(D2-Pad4)
- D8 pad 4: 5out -> in
- D80 pad 2: Net-(D80-Pad2) -> Net-(D2-Pad4)
- D80 pad 4: Net-(D72-Pad2) -> in
- D81 pad 2: Net-(D81-Pad2) -> Net-(D2-Pad4)
- D81 pad 4: Net-(D73-Pad2) -> in
- D82 pad 2: Net-(D82-Pad2) -> Net-(D2-Pad4)
- D82 pad 4: Net-(D74-Pad2) -> in
- D83 pad 2: Net-(D83-Pad2) -> Net-(D2-Pad4)
- D83 pad 4: Net-(D75-Pad2) -> in
- D84 pad 2: Net-(D84-Pad2) -> Net-(D2-Pad4)
- D84 pad 4: Net-(D76-Pad2) -> in
- D85 pad 2: Net-(D85-Pad2) -> Net-(D2-Pad4)
- D85 pad 4: Net-(D77-Pad2) -> in
- D86 pad 2: Net-(D86-Pad2) -> Net-(D2-Pad4)
- D86 pad 4: Net-(D78-Pad2) -> in
- D87 pad 2: Net-(D87-Pad2) -> Net-(D2-Pad4)
- D87 pad 4: Net-(D79-Pad2) -> in
- D88 pad 2: Net-(D88-Pad2) -> Net-(D2-Pad4)
- D88 pad 4: Net-(D80-Pad2) -> in
- D89 pad 2: Net-(D89-Pad2) -> Net-(D2-Pad4)
- D89 pad 4: Net-(D81-Pad2) -> in
- D9 pad 2: Net-(D17-Pad4) -> Net-(D2-Pad4)
- D9 pad 4: 6out -> in
- D90 pad 2: Net-(D90-Pad2) -> Net-(D2-Pad4)
- D90 pad 4: Net-(D82-Pad2) -> in
- D91 pad 2: 1out -> Net-(D2-Pad4)
- D91 pad 4: Net-(D83-Pad2) -> in
- D92 pad 2: 2out -> Net-(D2-Pad4)
- D92 pad 4: Net-(D84-Pad2) -> in
- D93 pad 2: 3out -> Net-(D2-Pad4)
- D93 pad 4: Net-(D85-Pad2) -> in
- D94 pad 2: 4out -> Net-(D2-Pad4)
- D94 pad 4: Net-(D86-Pad2) -> in
- D95 pad 2: 5out -> Net-(D2-Pad4)
- D95 pad 4: Net-(D87-Pad2) -> in
- D96 pad 2: 6out -> Net-(D2-Pad4)
- D96 pad 4: Net-(D88-Pad2) -> in
- D97 pad 1: +5V -> Net-(D97-Pad1)
- D97 pad 2: 7out -> +5V
- D98 pad 1: +5V -> Net-(D98-Pad1)
- D98 pad 2: unconnected-(D98-Pad2) -> VBUS
- JP17 pad 2: VCC -> VBUS
- R1 pad 2: CC1 -> Net-(D97-Pad1)
- R10 pad 1: PGND -> Net-(R10-Pad1)
- R2 pad 1: CC2 -> PGND
- R2 pad 2: PGND -> Net-(D98-Pad1)
- R3 pad 1: PGND -> Net-(R3-Pad1)
- R4 pad 1: Net-(R4-Pad1) -> PGND
- R4 pad 2: PGND -> CC1
- R6 pad 1: Net-(R6-Pad1) -> CC2
- R6 pad 2: Net-(D2-Pad1) -> PGND
- R7 pad 1: Net-(U10-Pad12) -> PGND
- R8 pad 1: Net-(U10-Pad13) -> Net-(R8-Pad1)
- R8 pad 2: Net-(D100-Pad1) (its old number) -> PGND
- R9 pad 1: PGND -> Net-(R9-Pad1)
- U1 pad 1: touch_state_3 -> touch_state_1
- U1 pad 3: touch_point_3 -> touch_point_1
- U10 pad 12: Net-(U10-Pad12) -> Net-(R9-Pad1)
- U10 pad 13: Net-(U10-Pad13) -> Net-(R10-Pad1)
- U2 pad 1: touch_state_4 -> touch_state_2
- U2 pad 3: touch_point_4 -> touch_point_2
- U3 pad 1: touch_state_1 -> touch_state_3
- U3 pad 3: touch_point_1 -> touch_point_3
- U4 pad 1: touch_state_2 -> touch_state_4
- U4 pad 3: touch_point_2 -> touch_point_4
- U6 pad 1: touch_state_7 -> touch_state_6
- U6 pad 3: touch_point_7 -> touch_point_6
- U6 pad 4: Net-(JP11-Pad1) -> Net-(JP12-Pad1)
- U6 pad 6: Net-(JP10-Pad1) -> Net-(JP11-Pad1)
- U7 pad 1: touch_state_8 -> touch_state_7
- U7 pad 3: touch_point_8 -> touch_point_7
- U7 pad 4: Net-(JP13-Pad1) -> Net-(JP14-Pad1)
- U7 pad 6: Net-(JP12-Pad1) -> Net-(JP13-Pad1)
- U8 pad 1: touch_state_5 -> touch_state_8
- U8 pad 3: touch_point_5 -> touch_point_8
- U8 pad 4: Net-(JP15-Pad1) -> Net-(JP16-Pad1)
- U8 pad 6: Net-(JP14-Pad1) -> Net-(JP15-Pad1)
Other:
- board size 149 x 107.8 mm -> 241.6 x 107.8 mm

Commit message: update
Parts:
- added U9: MAX77751CEFG_T, Snapeda:IC_MAX77751CEFG_T, F.Cu at (70.6, 159.2)
- moved R7 90.1 mm to (73.5, 167.2), turned to 180 degrees
- moved C19 85.5 mm to (76.2, 158.2), turned to -90 degrees
- moved R8 85.2 mm to (73.5, 165.1)
- moved C24 84.4 mm to (69.5, 163.0), turned to 180 degrees
- moved C18 80.0 mm to (74.0, 158.2), turned to -90 degrees
- moved C23 78.9 mm to (71.2, 153.6), turned to 180 degrees
- moved TP10 78.6 mm to (93.0, 162.8)
- moved C20 74.8 mm to (67.6, 155.8), turned to 180 degrees
- moved C25 64.9 mm to (78.4, 157.4), turned to 90 degrees
- moved C17 64.5 mm to (74.0, 161.8), turned to 90 degrees
- moved L1 60.2 mm to (76.4, 154.8)
- moved C21 55.2 mm to (74.2, 152.0), turned to 90 degrees
- moved TP9 53.4 mm to (86.8, 162.8)
- moved C22 41.2 mm to (71.2, 155.8), turned to 180 degrees
- moved D13 9.14 mm to (139.4, 66.4), turned to 180 degrees
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Connections:
- net Net-(C17-Pad2) renamed BAT
- net PGND renamed GND
- D1 pad 2: Net-(D2-Pad4) -> Net-(D1-Pad2)
- D10 pad 2: Net-(D2-Pad4) -> Net-(D10-Pad2)
- D10 pad 4: in -> Net-(D10-Pad4)
- D11 pad 2: Net-(D2-Pad4) -> Net-(D11-Pad2)
- D11 pad 4: in -> Net-(D10-Pad2)
- D12 pad 2: Net-(D2-Pad4) -> 1out
- D12 pad 4: in -> Net-(D11-Pad2)
- D13 pad 2: Net-(D2-Pad4) -> Net-(D13-Pad2)
- D13 pad 4: in -> 1out
- D14 pad 2: Net-(D2-Pad4) -> Net-(D14-Pad2)
- D14 pad 4: in -> Net-(D13-Pad2)
- D15 pad 2: Net-(D2-Pad4) -> Net-(D15-Pad2)
- D15 pad 4: in -> Net-(D14-Pad2)
- D16 pad 2: Net-(D2-Pad4) -> Net-(D16-Pad2)
- D16 pad 4: in -> Net-(D15-Pad2)
- D17 pad 2: Net-(D2-Pad4) -> Net-(D17-Pad2)
- D17 pad 4: in -> Net-(D16-Pad2)
- D18 pad 2: Net-(D2-Pad4) -> Net-(D18-Pad2)
- D18 pad 4: in -> Net-(D17-Pad2)
- D19 pad 2: Net-(D2-Pad4) -> Net-(D19-Pad2)
- D19 pad 4: in -> Net-(D18-Pad2)
- D2 pad 2: Net-(D2-Pad4) -> Net-(D2-Pad2)
- D2 pad 4: in -> Net-(D1-Pad2)
- D20 pad 2: Net-(D2-Pad4) -> Net-(D20-Pad2)
- D20 pad 4: in -> Net-(D19-Pad2)
- D21 pad 2: Net-(D2-Pad4) -> Net-(D21-Pad2)
- D21 pad 4: in -> Net-(D20-Pad2)
- D22 pad 2: Net-(D2-Pad4) -> Net-(D22-Pad2)
- D22 pad 4: in -> Net-(D21-Pad2)
- D23 pad 2: Net-(D2-Pad4) -> Net-(D23-Pad2)
- D23 pad 4: in -> Net-(D22-Pad2)
- D24 pad 2: Net-(D2-Pad4) -> 2out
- D24 pad 4: in -> Net-(D23-Pad2)
- D25 pad 2: Net-(D2-Pad4) -> Net-(D25-Pad2)
- D25 pad 4: in -> 2out
- D26 pad 2: Net-(D2-Pad4) -> Net-(D26-Pad2)
- D26 pad 4: in -> Net-(D25-Pad2)
- D27 pad 2: Net-(D2-Pad4) -> Net-(D27-Pad2)
- D27 pad 4: in -> Net-(D26-Pad2)
- D28 pad 2: Net-(D2-Pad4) -> Net-(D28-Pad2)
- D28 pad 4: in -> Net-(D27-Pad2)
- D29 pad 2: Net-(D2-Pad4) -> Net-(D29-Pad2)
- D29 pad 4: in -> Net-(D28-Pad2)
- D3 pad 2: Net-(D2-Pad4) -> Net-(D3-Pad2)
- D3 pad 4: in -> Net-(D2-Pad2)
- D30 pad 2: Net-(D2-Pad4) -> Net-(D30-Pad2)
- D30 pad 4: in -> Net-(D29-Pad2)
- D31 pad 2: Net-(D2-Pad4) -> Net-(D31-Pad2)
- D31 pad 4: in -> Net-(D30-Pad2)
- D32 pad 2: Net-(D2-Pad4) -> Net-(D32-Pad2)
- D32 pad 4: in -> Net-(D31-Pad2)
- D33 pad 2: Net-(D2-Pad4) -> Net-(D33-Pad2)
- D33 pad 4: in -> Net-(D32-Pad2)
- D34 pad 2: Net-(D2-Pad4) -> Net-(D34-Pad2)
- D34 pad 4: in -> Net-(D33-Pad2)
- D35 pad 2: Net-(D2-Pad4) -> Net-(D35-Pad2)
- D35 pad 4: in -> Net-(D34-Pad2)
- D36 pad 2: Net-(D2-Pad4) -> 3out
- D36 pad 4: in -> Net-(D35-Pad2)
- D37 pad 2: Net-(D2-Pad4) -> Net-(D37-Pad2)
- D37 pad 4: in -> 3out
- D38 pad 2: Net-(D2-Pad4) -> Net-(D38-Pad2)
- D38 pad 4: in -> Net-(D37-Pad2)
- D39 pad 2: Net-(D2-Pad4) -> Net-(D39-Pad2)
- D39 pad 4: in -> Net-(D38-Pad2)
- D4 pad 2: Net-(D2-Pad4) -> Net-(D4-Pad2)
- D4 pad 4: in -> Net-(D3-Pad2)
- D40 pad 2: Net-(D2-Pad4) -> Net-(D40-Pad2)
- D40 pad 4: in -> Net-(D39-Pad2)
- D41 pad 2: Net-(D2-Pad4) -> Net-(D41-Pad2)
- D41 pad 4: in -> Net-(D40-Pad2)
- D42 pad 2: Net-(D2-Pad4) -> Net-(D42-Pad2)
- D42 pad 4: in -> Net-(D41-Pad2)
- D43 pad 2: Net-(D2-Pad4) -> Net-(D43-Pad2)
- D43 pad 4: in -> Net-(D42-Pad2)
- D44 pad 2: Net-(D2-Pad4) -> Net-(D44-Pad2)
- D44 pad 4: in -> Net-(D43-Pad2)
- D45 pad 2: Net-(D2-Pad4) -> Net-(D45-Pad2)
- D45 pad 4: in -> Net-(D44-Pad2)
- D46 pad 2: Net-(D2-Pad4) -> Net-(D46-Pad2)
- D46 pad 4: in -> Net-(D45-Pad2)
- D47 pad 2: Net-(D2-Pad4) -> Net-(D47-Pad2)
- D47 pad 4: in -> Net-(D46-Pad2)
- D48 pad 2: Net-(D2-Pad4) -> 4out
- D48 pad 4: in -> Net-(D47-Pad2)
- D49 pad 2: Net-(D2-Pad4) -> Net-(D49-Pad2)
- D49 pad 4: in -> 4out
- D5 pad 2: Net-(D2-Pad4) -> Net-(D5-Pad2)
- D5 pad 4: in -> Net-(D4-Pad2)
- D50 pad 2: Net-(D2-Pad4) -> Net-(D50-Pad2)
- D50 pad 4: in -> Net-(D49-Pad2)
- D51 pad 2: Net-(D2-Pad4) -> Net-(D51-Pad2)
- D51 pad 4: in -> Net-(D50-Pad2)
- D52 pad 2: Net-(D2-Pad4) -> Net-(D52-Pad2)
- D52 pad 4: in -> Net-(D51-Pad2)
- D53 pad 2: Net-(D2-Pad4) -> Net-(D53-Pad2)
- D53 pad 4: in -> Net-(D52-Pad2)
- D54 pad 2: Net-(D2-Pad4) -> Net-(D54-Pad2)
- D54 pad 4: in -> Net-(D53-Pad2)
- D55 pad 2: Net-(D2-Pad4) -> Net-(D55-Pad2)
- D55 pad 4: in -> Net-(D54-Pad2)
- D56 pad 2: Net-(D2-Pad4) -> Net-(D56-Pad2)
- D56 pad 4: in -> Net-(D55-Pad2)
- D57 pad 2: Net-(D2-Pad4) -> Net-(D57-Pad2)
- D57 pad 4: in -> Net-(D56-Pad2)
- D58 pad 2: Net-(D2-Pad4) -> Net-(D58-Pad2)
- D58 pad 4: in -> Net-(D57-Pad2)
- D59 pad 2: Net-(D2-Pad4) -> Net-(D59-Pad2)
- D59 pad 4: in -> Net-(D58-Pad2)
- D6 pad 2: Net-(D2-Pad4) -> Net-(D6-Pad2)
- D6 pad 4: in -> Net-(D5-Pad2)
- D60 pad 2: Net-(D2-Pad4) -> 5out
- D60 pad 4: in -> Net-(D59-Pad2)
- D61 pad 2: Net-(D2-Pad4) -> Net-(D61-Pad2)
- D61 pad 4: in -> 5out
- D62 pad 2: Net-(D2-Pad4) -> Net-(D62-Pad2)
- D62 pad 4: in -> Net-(D61-Pad2)
- D63 pad 2: Net-(D2-Pad4) -> Net-(D63-Pad2)
- D63 pad 4: in -> Net-(D62-Pad2)
- D64 pad 2: Net-(D2-Pad4) -> Net-(D64-Pad2)
- D64 pad 4: in -> Net-(D63-Pad2)
- D65 pad 2: Net-(D2-Pad4) -> Net-(D65-Pad2)
- D65 pad 4: in -> Net-(D64-Pad2)
- D66 pad 2: Net-(D2-Pad4) -> Net-(D66-Pad2)
- D66 pad 4: in -> Net-(D65-Pad2)
- D67 pad 2: Net-(D2-Pad4) -> Net-(D67-Pad2)
- D67 pad 4: in -> Net-(D66-Pad2)
- D68 pad 2: Net-(D2-Pad4) -> Net-(D68-Pad2)
- D68 pad 4: in -> Net-(D67-Pad2)
- D69 pad 2: Net-(D2-Pad4) -> Net-(D69-Pad2)
- D69 pad 4: in -> Net-(D68-Pad2)
- D7 pad 2: Net-(D2-Pad4) -> Net-(D7-Pad2)
- D7 pad 4: in -> Net-(D6-Pad2)
- D70 pad 2: Net-(D2-Pad4) -> Net-(D70-Pad2)
- D70 pad 4: in -> Net-(D69-Pad2)
- D71 pad 2: Net-(D2-Pad4) -> Net-(D71-Pad2)
- D71 pad 4: in -> Net-(D70-Pad2)
- D72 pad 2: Net-(D2-Pad4) -> 6out
- D72 pad 4: in -> Net-(D71-Pad2)
- D73 pad 2: Net-(D2-Pad4) -> Net-(D73-Pad2)
- D73 pad 4: in -> 6out
- D74 pad 2: Net-(D2-Pad4) -> Net-(D74-Pad2)
- D74 pad 4: in -> Net-(D73-Pad2)
- D75 pad 2: Net-(D2-Pad4) -> Net-(D75-Pad2)
- D75 pad 4: in -> Net-(D74-Pad2)
- D76 pad 2: Net-(D2-Pad4) -> Net-(D76-Pad2)
- D76 pad 4: in -> Net-(D75-Pad2)
- D77 pad 2: Net-(D2-Pad4) -> Net-(D77-Pad2)
- D77 pad 4: in -> Net-(D76-Pad2)
- D78 pad 2: Net-(D2-Pad4) -> Net-(D78-Pad2)
- D78 pad 4: in -> Net-(D77-Pad2)
- D79 pad 2: Net-(D2-Pad4) -> Net-(D79-Pad2)
- D79 pad 4: in -> Net-(D78-Pad2)
- D8 pad 2: Net-(D2-Pad4) -> Net-(D8-Pad2)
- D8 pad 4: in -> Net-(D7-Pad2)
- D80 pad 2: Net-(D2-Pad4) -> Net-(D80-Pad2)
- D80 pad 4: in -> Net-(D79-Pad2)
- D81 pad 2: Net-(D2-Pad4) -> Net-(D81-Pad2)
- D81 pad 4: in -> Net-(D80-Pad2)
- D82 pad 2: Net-(D2-Pad4) -> Net-(D82-Pad2)
- D82 pad 4: in -> Net-(D81-Pad2)
- D83 pad 2: Net-(D2-Pad4) -> Net-(D83-Pad2)
- D83 pad 4: in -> Net-(D82-Pad2)
- D84 pad 2: Net-(D2-Pad4) -> 7out
- D84 pad 4: in -> Net-(D83-Pad2)
- D85 pad 2: Net-(D2-Pad4) -> Net-(D85-Pad2)
- D85 pad 4: in -> 7out
- D86 pad 2: Net-(D2-Pad4) -> Net-(D86-Pad2)
- D86 pad 4: in -> Net-(D85-Pad2)
- D87 pad 2: Net-(D2-Pad4) -> Net-(D87-Pad2)
- D87 pad 4: in -> Net-(D86-Pad2)
- D88 pad 2: Net-(D2-Pad4) -> Net-(D88-Pad2)
- D88 pad 4: in -> Net-(D87-Pad2)
- D89 pad 2: Net-(D2-Pad4) -> Net-(D89-Pad2)
- D89 pad 4: in -> Net-(D88-Pad2)
- D9 pad 2: Net-(D2-Pad4) -> Net-(D10-Pad4)
- D9 pad 4: in -> Net-(D8-Pad2)
- D90 pad 2: Net-(D2-Pad4) -> Net-(D90-Pad2)
- D90 pad 4: in -> Net-(D89-Pad2)
- D91 pad 2: Net-(D2-Pad4) -> Net-(D91-Pad2)
- D91 pad 4: in -> Net-(D90-Pad2)
- D92 pad 2: Net-(D2-Pad4) -> Net-(D92-Pad2)
- D92 pad 4: in -> Net-(D91-Pad2)
- D93 pad 2: Net-(D2-Pad4) -> Net-(D93-Pad2)
- D93 pad 4: in -> Net-(D92-Pad2)
- D94 pad 2: Net-(D2-Pad4) -> Net-(D94-Pad2)
- D94 pad 4: in -> Net-(D93-Pad2)
- D95 pad 2: Net-(D2-Pad4) -> Net-(D95-Pad2)
- D95 pad 4: in -> Net-(D94-Pad2)
- D96 pad 2: Net-(D2-Pad4) -> unconnected-(D96-Pad2)
- D96 pad 4: in -> Net-(D95-Pad2)
- L1 pad 2: SYS -> +5V
Routing:
- net BST: track 0.00 -> 0.57 mm, vias 0 -> 1
- net LX: vias 0 -> 5
- added copper zone on F.Cu, net +5V
- added copper zone on B.Cu, net LX
- added copper zone on F.Cu, net LX

Commit message: Update design.kicad_pcb
Parts:
- moved J1 97.7 mm to (45.5, 159.6), turned to -90 degrees
- moved D100 71.9 mm to (63.0, 149.1), turned to 90 degrees
- moved R3 42.6 mm to (60.7, 152.9), turned to 90 degrees
- moved R5 42.5 mm to (63.0, 152.9), turned to 90 degrees
- moved D99 36.8 mm to (60.7, 149.1), turned to 90 degrees
- moved TP9 4.01 mm to (90.8, 162.8)
- moved TP10 3.93 mm to (96.9, 162.8)
- moved R7 2.13 mm to (73.5, 165.1)
- moved R8 2.07 mm to (73.5, 167.2)
Routing:
- net VBUS: track 0.00 -> 30.3 mm, vias 0 -> 2
- net D-: track 0.00 -> 26.8 mm
- net D+: track 0.00 -> 25.5 mm, vias 0 -> 2
- net CC2: track 0.00 -> 19.8 mm, vias 0 -> 2
- net CC1: track 0.00 -> 19.4 mm
- net Net-(R3-Pad1): track 0.00 -> 11.5 mm, vias 0 -> 2
- net BST: track 0.57 -> 10.5 mm, vias 1 -> 2
- net Net-(R5-Pad1): track 0.00 -> 9.32 mm, vias 0 -> 2
- net Net-(R8-Pad1): track 0.00 -> 7.52 mm
- net Net-(R7-Pad2): track 0.00 -> 5.12 mm
- net BYP: track 0.00 -> 4.16 mm
- net Net-(JP17-Pad1): track 0.00 -> 2.27 mm
- net BAT: track 0.00 -> 2.23 mm, vias 0 -> 4
- net VDD: track 0.00 -> 2.17 mm
- net Net-(D99-Pad1): track 0.00 -> 2.11 mm
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- added copper zone on B.Cu, net BAT
- added copper zone on F.Cu, net BAT
- added copper zone on F.Cu, net GND
Other:
- board size 241.6 x 107.8 mm -> 241.6 x 144.1 mm

Commit message: Update design.kicad_pcb
Parts:
- C1, C10, C11, C12, C13, C14, C15, C16, C17, C18, C19, C2, C20, C21, C22, C23, C24, C25, C26, C27, C3, C4, C5, C6, C7, C8, C9, D100, D99, J1, JP1, JP10, JP11, JP12, JP13, JP14, JP15, JP16, JP17, JP2, JP3, JP4, JP5, JP6, JP7, JP8, JP9, L1, R3, R4, R5, R6, R7, R8, TP10, TP9, U1, U10, U2, U3, U4, U5, U6, U7, U8, U9: moved to B.Cu
- moved C11 208.2 mm to (228.0, 131.8), turned to 90 degrees
- moved JP15 207.6 mm to (235.8, 128.7), turned to 180 degrees
- moved C12 197.0 mm to (242.4, 132.0), turned to 90 degrees
- moved C10 190.6 mm to (214.4, 132.0), turned to 90 degrees
- moved U7 188.5 mm to (224.2, 131.8), turned to 180 degrees
- moved JP11 187.4 mm to (207.8, 128.7), turned to 180 degrees
- moved JP14 185.2 mm to (221.4, 135.1), turned to 180 degrees
- moved JP12 184.4 mm to (207.8, 135.3), turned to 180 degrees
- moved JP13 184.2 mm to (221.4, 128.5), turned to 180 degrees
- moved U5 180.2 mm to (196.7, 131.8), turned to 180 degrees
- moved U6 179.7 mm to (210.4, 132.0), turned to 180 degrees
- moved U8 174.9 mm to (238.4, 132.0), turned to 180 degrees
- moved C15 174.8 mm to (219.6, 131.8), turned to 180 degrees
- moved JP16 166.4 mm to (235.8, 135.3), turned to 180 degrees
- moved C14 166.1 mm to (205.7, 132.0), turned to 180 degrees
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Routing:
- net VCC: track 0.00 -> 75.6 mm
- net GND: track 1.52 -> 30.5 mm
- net CC1: track 19.4 -> 26.5 mm
- net CC2: track 19.8 -> 25.8 mm
- net Net-(JP10-Pad1): track 0.00 -> 3.02 mm
- net Net-(JP9-Pad1): track 0.00 -> 3.02 mm
- net touch_point_8: track 0.00 -> 2.93 mm
- net touch_point_5: track 0.00 -> 2.93 mm
- net touch_point_4: track 0.00 -> 2.93 mm
- net touch_point_2: track 0.00 -> 2.93 mm
- net touch_point_1: track 0.00 -> 2.93 mm
- net touch_point_6: track 0.00 -> 2.79 mm
- net Net-(JP8-Pad1): track 0.00 -> 2.77 mm
- net Net-(JP7-Pad1): track 0.00 -> 2.77 mm
- net Net-(JP13-Pad1): track 0.00 -> 2.77 mm
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- added copper zone on B.Cu, net +5V
- added copper zone on B.Cu, net GND
- removed copper zone on F.Cu, net +5V
- removed copper zone on F.Cu, net GND
Other:
- board size 241.6 x 144.1 mm -> 136.2 x 88.1 mm
