File: design.kicad_pcb (KiCad board)
At the start: 2 copper layers, 122.6 x 97.8 mm, 156 parts, among them J301 TYPE-C-31-M-12, U1 TTP223, U10 ATtiny1616-M, U2 TTP223, U3 TTP223, U4 TTP223, U5 TTP223, U6 TTP223, U7 TTP223, U8 TTP223

Commit message: Update design.kicad_pcb
Routing:
- net unconnected-(J301-PadS1): track 17.0 -> 0.00 mm
Changed lines of the file:
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@@
     (fp_circle (center -3.2 6) (end -3.1 6) (layer "B.SilkS") (width 0.2) (fill none))
+    (fp_poly (pts
+        (xy 1.55 5.37)
+        (xy 1.95 5.37)
+        (xy 1.95 4.13)
+        (xy 1.55 4.13)
+      ) (layer "B.Mask") (width 0.01) (fill solid))
+    (fp_poly (pts
+        (xy -0.95 5.37)
+        (xy -0.55 5.37)
+        (xy -0.55 4.13)
+        (xy -0.95 4.13)
+      ) (layer "B.Mask") (width 0.01) (fill solid))
     (fp_poly (pts
         (xy 0.05 5.37)
@@
       ) (layer "B.Mask") (width 0.01) (fill solid))
     (fp_poly (pts
-        (xy 1.55 5.37)
-        (xy 1.95 5.37)
-        (xy 1.95 4.13)
-        (xy 1.55 4.13)
+        (xy 2.85 5.37)
+        (xy 3.55 5.37)
+        (xy 3.55 4.13)
+        (xy 2.85 4.13)
+      ) (layer "B.Mask") (width 0.01) (fill solid))
+    (fp_poly (pts
+        (xy -1.95 5.37)
+        (xy -1.55 5.37)
+        (xy -1.55 4.13)
+        (xy -1.95 4.13)
+      ) (layer "B.Mask") (width 0.01) (fill solid))
+    (fp_poly (pts
+        (xy -3.55 5.37)
+        (xy -2.85 5.37)
+        (xy -2.85 4.13)
+        (xy -3.55 4.13)
+      ) (layer "B.Mask") (width 0.01) (fill solid))
+    (fp_poly (pts
+        (xy 1.05 5.37)
+        (xy 1.45 5.37)
+        (xy 1.45 4.13)
+        (xy 1.05 4.13)
       ) (layer "B.Mask") (width 0.01) (fill solid))
     (fp_poly (pts
@@
       ) (layer "B.Mask") (width 0.01) (fill solid))
     (fp_poly (pts
-        (xy -2.75 5.37)
-        (xy -2.05 5.37)
-        (xy -2.05 4.13)
-        (xy -2.75 4.13)
+        (xy 0.55 5.37)
+        (xy 0.95 5.37)
+        (xy 0.95 4.13)
+        (xy 0.55 4.13)
       ) (layer "B.Mask") (width 0.01) (fill solid))
     (fp_poly (pts
@@
       ) (layer "B.Mask") (width 0.01) (fill solid))
     (fp_poly (pts
-        (xy -1.95 5.37)
-        (xy -1.55 5.37)
-        (xy -1.55 4.13)
-        (xy -1.95 4.13)
+        (xy -2.75 5.37)
+        (xy -2.05 5.37)
+        (xy -2.05 4.13)
+        (xy -2.75 4.13)
       ) (layer "B.Mask") (width 0.01) (fill solid))
-    (fp_poly (pts
-        (xy 2.85 5.37)
-        (xy 3.55 5.37)
-        (xy 3.55 4.13)
-        (xy 2.85 4.13)
-      ) (layer "B.Mask") (width 0.01) (fill solid))
-    (fp_poly (pts
-        (xy -3.55 5.37)
-        (xy -2.85 5.37)
-        (xy -2.85 4.13)
-        (xy -3.55 4.13)
-      ) (layer "B.Mask") (width 0.01) (fill solid))
-    (fp_poly (pts
-        (xy 0.55 5.37)
-        (xy 0.95 5.37)
-        (xy 0.95 4.13)
-        (xy 0.55 4.13)
-      ) (layer "B.Mask") (width 0.01) (fill solid))
-    (fp_poly (pts
-        (xy -0.95 5.37)
-        (xy -0.55 5.37)
-        (xy -0.55 4.13)
-        (xy -0.95 4.13)
-      ) (layer "B.Mask") (width 0.01) (fill solid))
-    (fp_poly (pts
-        (xy 1.05 5.37)
-        (xy 1.45 5.37)
-        (xy 1.45 4.13)
-        (xy 1.05 4.13)
-      ) (layer "B.Mask") (width 0.01) (fill solid))
+    (fp_line (start -5.025 -2.85) (end 5.025 -2.85) (layer "B.CrtYd") (width 0.05))
+    (fp_line (start -5.025 5.57) (end -5.025 -2.85) (layer "B.CrtYd") (width 0.05))
     (fp_line (start 5.025 5.57) (end -5.025 5.57) (layer "B.CrtYd") (width 0.05))
-    (fp_line (start -5.025 -2.85) (end 5.025 -2.85) (layer "B.CrtYd") (width 0.05))
     (fp_line (start 5.025 -2.85) (end 5.025 5.57) (layer "B.CrtYd") (width 0.05))
-    (fp_line (start -5.025 5.57) (end -5.025 -2.85) (layer "B.CrtYd") (width 0.05))
     (fp_line (start -5.5 -2.11) (end 9 -2.11) (layer "B.Fab") (width 0.127))
-    (fp_line (start 4.47 -2.6) (end 4.47 4.75) (layer "B.Fab") (width 0.127))
-    (fp_line (start -4.47 4.75) (end -4.47 -2.6) (layer "B.Fab") (width 0.127))
     (fp_line (start -4.47 -2.6) (end 4.47 -2.6) (layer "B.Fab") (width 0.127))
-    (fp_line (start 4.47 -2.6) (end 4.47 -1.17) (layer "B.Fab") (width 0.127))
     (fp_line (start -4.47 -2.6) (end 4.47 -2.6) (layer "B.Fab") (width 0.127))
     (fp_line (start -4.47 -2.6) (end -4.47 -1.17) (layer "B.Fab") (width 0.127))
     (fp_line (start 4.47 4.75) (end -4.47 4.75) (layer "B.Fab") (width 0.127))
+    (fp_line (start 4.47 -2.6) (end 4.47 4.75) (layer "B.Fab") (width 0.127))
+    (fp_line (start 4.47 -2.6) (end 4.47 -1.17) (layer "B.Fab") (width 0.127))
+    (fp_line (start -4.47 4.75) (end -4.47 -2.6) (layer "B.Fab") (width 0.127))
     (fp_circle (center -3.2 6) (end -3.1 6) (layer "B.Fab") (width 0.2) (fill none))
     (pad "" np_thru_hole circle (at -2.89 3.68 90) (size 0.6 0.6) (drill 0.6) (layers *.Cu *.Mask))
@@
     (pad "B8" smd rect (at -1.75 4.75 90) (size 0.3 1.14) (layers "B.Cu" "B.Paste")
       (net 152 "unconnected-(J301-PadB8)") (pinfunction "SBU2") (pintype "bidirectional+no_connect"))
+    (pad "S1" thru_hole oval (at 4.325 0 90) (size 0.9 1.7) (drill oval 0.6 1.4) (layers *.Cu *.Mask)
+      (net 153 "unconnected-(J301-PadS1)") (pinfunction "SHIELD") (pintype "passive+no_connect") (solder_mask_margin 0.102))
+    (pad "S1" thru_hole oval (at -4.325 0 90) (size 0.9 1.7) (drill oval 0.6 1.4) (layers *.Cu *.Mask)
+      (net 153 "unconnected-(J301-PadS1)") (pinfunction "SHIELD") (pintype "passive+no_connect") (solder_mask_margin 0.102))
+    (pad "S1" thru_hole oval (at 4.325 4.17 90) (size 0.9 2) (drill oval 0.6 1.7) (layers *.Cu *.Mask)
+      (net 153 "unconnected-(J301-PadS1)") (pinfunction "SHIELD") (pintype "passive+no_connect") (solder_mask_margin 0.102))
     (pad "S1" thru_hole oval (at -4.325 4.17 90) (size 0.9 2) (drill oval 0.6 1.7) (layers *.Cu *.Mask)
-      (net 153 "unconnected-(J301-PadS1)") (pinfunction "SHIELD") (pintype "passive+no_connect") (solder_mask_margin 0.102))
-    (pad "S2" thru_hole oval (at 4.325 4.17 90) (size 0.9 2) (drill oval 0.6 1.7) (layers *.Cu *.Mask)
-      (net 153 "unconnected-(J301-PadS1)") (pinfunction "SHIELD") (pintype "passive+no_connect") (solder_mask_margin 0.102))
-    (pad "S3" thru_hole oval (at -4.325 0 90) (size 0.9 1.7) (drill oval 0.6 1.4) (layers *.Cu *.Mask)
-      (net 153 "unconnected-(J301-PadS1)") (pinfunction "SHIELD") (pintype "passive+no_connect") (solder_mask_margin 0.102))
-    (pad "S4" thru_hole oval (at 4.325 0 90) (size 0.9 1.7) (drill oval 0.6 1.4) (layers *.Cu *.Mask)
       (net 153 "unconnected-(J301-PadS1)") (pinfunction "SHIELD") (pintype "passive+no_connect") (solder_mask_margin 0.102))
     (model "${KICAD_3RD_PARTY}/Snapeda.3dshapes/TYPE-C-31-M-12.step"
@@
   (segment (start 130.475 128.175) (end 131.05 128.75) (width 0.21) (layer "B.Cu") (net 149))
   (segment (start 130.475 124.4) (end 130.475 128.175) (width 0.21) (layer "B.Cu") (net 149))
-  (segment (start 128.48 134.825) (end 128.48 126.175) (width 0.25) (layer "F.Cu") (net 153))
-  (segment (start 128.48 126.175) (end 132.65 126.175) (width 0.25) (layer "F.Cu") (net 153))
-  (segment (start 128.48 134.825) (end 132.65 134.825) (width 0.25) (layer "F.Cu") (net 153))
   (zone (net 8) (net_name "touch_point_8") (layer "F.Cu") (hatch edge 0.508)
     (priority 1)
