File: design.kicad_sch (KiCad schematic)
At the start: 14 parts, among them J1 Conn_01x02, J2 Conn_01x02, J3 Conn_01x03, J4 Conn_01x03, U1 TPS61099YFFT

Commit message: Update design.kicad_sch
Parts:
- removed C1, C2, C3, C4: C_Small, Capacitor_SMD:C_0805_2012Metric, symbol Device:C_Small
- removed J1, J2: Conn_01x02, Connector_PinHeader_2.54mm:PinHeader_1x02_P2.54mm_Vertical, symbol Connector_Generic:Conn_01x02
- removed J3, J4: Conn_01x03, Connector_PinHeader_2.54mm:PinHeader_1x03_P2.54mm_Vertical, symbol Connector_Generic:Conn_01x03
- removed JP1, JP2: SolderJumper_2_Open, Jumper:SolderJumper-2_P1.3mm_Open_RoundedPad1.0x1.5mm, symbol Jumper:SolderJumper_2_Open
- removed L1: L_Small, Inductor_SMD:L_1008_2520Metric, symbol Device:L_Small
- removed R1, R2: R_Small, Resistor_SMD:R_0805_2012Metric, symbol Device:R_Small
- removed U1: TPS61099YFFT, Converter_DCDC_custom:BGA6N40P3X2_122X88X62N, symbol Converter_DCDC_custom:TPS61099YFFT
- added C? (x8): 0-50pF, Capacitor_SMD:C_0805_2012Metric, symbol Device:C_Small
- added C? (x2): C_Small, symbol Device:C_Small
- added C? (x8): 100nF, Capacitor_SMD:C_0805_2012Metric, symbol Device:C_Small
- added D? (x96): WS2812B, LED_SMD:LED_WS2812B_PLCC4_5.0x5.0mm_P3.2mm, symbol LED:WS2812B
- added JP? (x8): AHLB, Jumper:SolderJumper-2_P1.3mm_Open_RoundedPad1.0x1.5mm, symbol Jumper:Jumper_2_Open
- added JP? (x8): TOG, Jumper:SolderJumper-2_P1.3mm_Open_RoundedPad1.0x1.5mm, symbol Jumper:Jumper_2_Open
- added TP? (x8): touch_point_2, symbol Connector:TestPoint
- added U? (x8): TTP223, Package_TO_SOT_SMD:SOT-23-6_Handsoldering, symbol LEDs:TTP223
- added U?: MAX77751CEFG_T, Snapeda:MAX77751CEFG_T_IC_MAX77751CEFG_T, symbol Snapeda:MAX77751CEFG_T
- added U?: ATtiny1616-S, Package_SO:SOIC-20W_7.5x12.8mm_P1.27mm, symbol MCU_Microchip_ATtiny:ATtiny1616-S
Connections:
- net GND: now also C?.2, C?.2, C?.2, C?.2, C?.2, C?.2, C?.2, C?.2, C?.2, C?.2, C?.2, C?.2, C?.2, C?.2, C?.2, C?.2, C?.2, C?.2, D?.3 (VSS), D?.3 (VSS), D?.3 (VSS), D?.3 (VSS), D?.3 (VSS), D?.3 (VSS), D?.3 (VSS), D?.3 (VSS), D?.3 (VSS), D?.3 (VSS), D?.3 (VSS), D?.3 (VSS), D?.3 (VSS), D?.3 (VSS), D?.3 (VSS), D?.3 (VSS), D?.3 (VSS), D?.3 (VSS), D?.3 (VSS), D?.3 (VSS), D?.3 (VSS), D?.3 (VSS), D?.3 (VSS), D?.3 (VSS), D?.3 (VSS), D?.3 (VSS), D?.3 (VSS), D?.3 (VSS), D?.3 (VSS), D?.3 (VSS), D?.3 (VSS), D?.3 (VSS), D?.3 (VSS), D?.3 (VSS), D?.3 (VSS), D?.3 (VSS), D?.3 (VSS), D?.3 (VSS), D?.3 (VSS), D?.3 (VSS), D?.3 (VSS), D?.3 (VSS), D?.3 (VSS), D?.3 (VSS), D?.3 (VSS), D?.3 (VSS), D?.3 (VSS), D?.3 (VSS), D?.3 (VSS), D?.3 (VSS), D?.3 (VSS), D?.3 (VSS), D?.3 (VSS), D?.3 (VSS), D?.3 (VSS), D?.3 (VSS), D?.3 (VSS), D?.3 (VSS), D?.3 (VSS), D?.3 (VSS), D?.3 (VSS), D?.3 (VSS), D?.3 (VSS), D?.3 (VSS), D?.3 (VSS), D?.3 (VSS), D?.3 (VSS), D?.3 (VSS), D?.3 (VSS), D?.3 (VSS), D?.3 (VSS), D?.3 (VSS), D?.3 (VSS), D?.3 (VSS), D?.3 (VSS), D?.3 (VSS), D?.3 (VSS), D?.3 (VSS), D?.3 (VSS), D?.3 (VSS), D?.3 (VSS), D?.3 (VSS), D?.3 (VSS), D?.3 (VSS), D?.3 (VSS), D?.3 (VSS), D?.3 (VSS), D?.3 (VSS), D?.3 (VSS), D?.3 (VSS), D?.3 (VSS), D?.3 (VSS), D?.3 (VSS), D?.3 (VSS), D?.3 (VSS), D?.3 (VSS), U?.2 (GND), U?.2 (GND), U?.2 (GND), U?.2 (GND), U?.2 (GND), U?.2 (GND), U?.2 (GND), U?.2 (GND), U?.20 (GND)
- new net: D?.2 (DOUT), D?.4 (DIN) (x88)
- new net: JP?.1 (A), U?.4 (AHLB) (x8)
- new net: JP?.1 (A), U?.6 (TOG) (x8)
- new net +5V: C?.1, C?.1, D?.1 (VDD), D?.1 (VDD), D?.1 (VDD), D?.1 (VDD), D?.1 (VDD), D?.1 (VDD), D?.1 (VDD), D?.1 (VDD), D?.1 (VDD), D?.1 (VDD), D?.1 (VDD), D?.1 (VDD), D?.1 (VDD), D?.1 (VDD), D?.1 (VDD), D?.1 (VDD), D?.1 (VDD), D?.1 (VDD), D?.1 (VDD), D?.1 (VDD), D?.1 (VDD), D?.1 (VDD), D?.1 (VDD), D?.1 (VDD), D?.1 (VDD), D?.1 (VDD), D?.1 (VDD), D?.1 (VDD), D?.1 (VDD), D?.1 (VDD), D?.1 (VDD), D?.1 (VDD), D?.1 (VDD), D?.1 (VDD), D?.1 (VDD), D?.1 (VDD), D?.1 (VDD), D?.1 (VDD), D?.1 (VDD), D?.1 (VDD), D?.1 (VDD), D?.1 (VDD), D?.1 (VDD), D?.1 (VDD), D?.1 (VDD), D?.1 (VDD), D?.1 (VDD), D?.1 (VDD), D?.1 (VDD), D?.1 (VDD), D?.1 (VDD), D?.1 (VDD), D?.1 (VDD), D?.1 (VDD), D?.1 (VDD), D?.1 (VDD), D?.1 (VDD), D?.1 (VDD), D?.1 (VDD), D?.1 (VDD), D?.1 (VDD), D?.1 (VDD), D?.1 (VDD), D?.1 (VDD), D?.1 (VDD), D?.1 (VDD), D?.1 (VDD), D?.1 (VDD), D?.1 (VDD), D?.1 (VDD), D?.1 (VDD), D?.1 (VDD), D?.1 (VDD), D?.1 (VDD), D?.1 (VDD), D?.1 (VDD), D?.1 (VDD), D?.1 (VDD), D?.1 (VDD), D?.1 (VDD), D?.1 (VDD), D?.1 (VDD), D?.1 (VDD), D?.1 (VDD), D?.1 (VDD), D?.1 (VDD), D?.1 (VDD), D?.1 (VDD), D?.1 (VDD), D?.1 (VDD), D?.1 (VDD), D?.1 (VDD), D?.1 (VDD), D?.1 (VDD), D?.1 (VDD), D?.1 (VDD), U?.1 (VCC)
- new net 1out: D?.2 (DOUT), D?.4 (DIN)
- new net 2out: D?.2 (DOUT), D?.4 (DIN)
- new net 3out: D?.2 (DOUT), D?.4 (DIN)
- new net 4out: D?.2 (DOUT), D?.4 (DIN)
- new net 5out: D?.2 (DOUT), D?.4 (DIN)
- new net 6out: D?.2 (DOUT), D?.4 (DIN)
- new net 7out: D?.2 (DOUT), D?.4 (DIN)
- new net UPDI: U?.16 (~{RESET}/PA0)
- new net VCC: C?.1, C?.1, C?.1, C?.1, C?.1, C?.1, C?.1, C?.1, JP?.2 (B), JP?.2 (B), JP?.2 (B), JP?.2 (B), JP?.2 (B), JP?.2 (B), JP?.2 (B), JP?.2 (B), JP?.2 (B), JP?.2 (B), JP?.2 (B), JP?.2 (B), JP?.2 (B), JP?.2 (B), JP?.2 (B), JP?.2 (B), U?.5 (VCC), U?.5 (VCC), U?.5 (VCC), U?.5 (VCC), U?.5 (VCC), U?.5 (VCC), U?.5 (VCC), U?.5 (VCC)
- new net in: D?.4 (DIN), U?.18 (PA2)
- new net touch_point_1: C?.1, TP?.1, U?.3 (I), U?.4 (PA6)
- new net touch_point_2: C?.1, TP?.1, U?.3 (I), U?.5 (PA7)
- new net touch_point_3: C?.1, TP?.1, U?.11 (PB0), U?.3 (I)
- new net touch_point_4: C?.1, TP?.1, U?.10 (PB1), U?.3 (I)
- new net touch_point_5: C?.1, TP?.1, U?.3 (I), U?.9 (PB2)
- new net touch_point_6: C?.1, TP?.1, U?.3 (I), U?.8 (PB3)
- new net touch_point_7: C?.1, TP?.1, U?.3 (I), U?.7 (PB4)
- new net touch_point_8: C?.1, TP?.1, U?.3 (I), U?.6 (PB5)
- new net touch_state_1: U?.1 (Q)
- new net touch_state_2: U?.1 (Q)
- new net touch_state_3: U?.1 (Q)
- new net touch_state_4: U?.1 (Q)
- new net touch_state_5: U?.1 (Q)
- new net touch_state_6: U?.1 (Q)
- new net touch_state_7: U?.1 (Q)
- new net touch_state_8: U?.1 (Q)
- no-connect marks 0 -> 8
Other:
- note added: "TOG: LOW - Direct Mode HIGH - Toggle Mode AHLB: LOW - CMOS active high output HIGH - CMOS active low output"

Commit message: Update design.kicad_sch
Parts:
- added C?: 22uF, symbol Device:C_Small
- added C? (x4): 10uF, symbol Device:C_Small
- added C? (x3): 2.2uF, symbol Device:C_Small
- added C?: 0.1uF, symbol Device:C_Small
- added D? (x2): LED_Small, symbol Device:LED_Small
- added J?: TYPE-C-31-M-12, Snapeda:TYPE-C-31-M-12_HRO_TYPE-C-31-M-12, symbol Snapeda:TYPE-C-31-M-12
- added JP?: ENBST, symbol Jumper:Jumper_2_Bridged
- added L?: 0.47uH, symbol Device:L_Small
- added R?: 13.3k, Resistor_SMD:R_0805_2012Metric, symbol Device:R_Small
- added R?: 2.4k, Resistor_SMD:R_0805_2012Metric, symbol Device:R_Small
- added R? (x2): 1k, Resistor_SMD:R_0805_2012Metric, symbol Device:R_Small
- added R? (x2): 5.1k, Resistor_SMD:R_0805_2012Metric, symbol Device:R_Small
- added TP?: BAT-, symbol Connector:TestPoint
- added TP?: BAT+, symbol Connector:TestPoint
Connections:
- net +5V: now also U?.15_16 (SYS), C?.2, C?.2, D?.2 (A), D?.2 (A)
- net GND: now also U?.18_19 (PGND), U?.9 (GND), C?.1, C?.1, C?.1, C?.1, C?.1, C?.2, C?.2, C?.2, J?.A1_B12 (GND), J?.B1_A12 (GND), R?.1, R?.1, R?.2, R?.2, TP?.1
- net BST: now reaches U?.1 (BST)
- net BST: now also C?.2
- net VDD: now reaches U?.10 (VDD)
- net VDD: now also C?.1
- net at U?.11 (ITOPOFF): now also R?.1
- net at U?.12 (IFAST): now also R?.2
- net at U?.13_14 (BATT): now also C?.2, TP?.1
- net PVL: now reaches U?.17 (PVL)
- net PVL: now also C?.1
- net at U?.2 (INOKB): now also R?.1
- net LX: now reaches U?.20_21 (LX)
- net LX: now also C?.1, L?.1
- net BYP: now reaches U?.22 (BYP)
- net BYP: now also C?.2, C?.2
- net VBUS: now reaches U?.23_24 (CHGIN)
- net VBUS: now also C?.1, J?.A4_B9 (VBUS), J?.B4_A9 (VBUS), JP?.2 (B)
- net at U?.3 (STAT): now also R?.1
- net CC2: now reaches U?.4 (CC2)
- net CC2: now also J?.B5 (CC2), R?.1
- net CC1: now reaches U?.5 (CC1)
- net CC1: now also J?.A5 (CC1), R?.2
- net D+: now reaches U?.6 (DP)
- net D+: now also J?.A6 (DP1), J?.B6 (DP2)
- net D-: now reaches U?.7 (DN)
- net D-: now also J?.A7 (DN1), J?.B7 (DN2)
- net at U?.8 (ENBST): now also JP?.1 (A)
- new net: D?.1 (K), R?.2 (x2)
- new net: J?.S1 (SHIELD), J?.S2 (SHIELD), J?.S3 (SHIELD), J?.S4 (SHIELD)
- new net SYS: L?.2
- no-connect marks 8 -> 11
Other:
- note added: "If ENBST is driven high, the reverse boost is enabled and the BYP-to-CHGIN path is closed. internall pulldown"
- moved on the sheet: C?, U?

Commit message: Update design.kicad_sch
Parts:
- added D100, D99: LED_Small, symbol Device:LED_Small
- added R7, R8: 1k, Resistor_SMD:R_0805_2012Metric, symbol Device:R_Small
- gave numbers to parts that had none: 170
Connections:
- net +5V: now also D100.2 (A), D99.2 (A)
- net at U10.12 (PC0): now also R7.1
- net at U10.13 (PC1): now also R8.1
- new net: D99.1 (K), R7.2
- new net: D100.1 (K), R8.2
- no-connect marks 11 -> 9
Other:
- note added: "RESISTANCE (kΩ) IFAST (mA) 2.4 500 RTOPOFF (kΩ) ITOPOFF (mA) 13.3 200"
- moved on the sheet: C22, C24

Commit message: Update design.kicad_sch
Parts:
- added D? (x2): LED_Small, symbol Device:LED_Small
- added R? (x2): 1k, Resistor_SMD:R_0805_2012Metric, symbol Device:R_Small
Connections:
- net +5V: now also D?.2 (A)
- net GND: now also R?.1, R?.1
- net VBUS: now also D?.2 (A)
- new net: D?.1 (K), R?.2 (x2)
Changed lines of the file:
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@@
     (stroke (width 0) (type default) (color 0 0 0 0))
   )
+  (wire (pts (xy 88.9 64.77) (xy 88.9 61.595))
+    (stroke (width 0) (type default) (color 0 0 0 0))
+  )
   (wire (pts (xy 85.852 239.395) (xy 88.392 239.395))
     (stroke (width 0) (type default) (color 0 0 0 0))
@@
     (stroke (width 0) (type default) (color 0 0 0 0))
   )
+  (wire (pts (xy 231.14 47.625) (xy 231.14 43.18))
+    (stroke (width 0) (type default) (color 0 0 0 0))
+  )
   (wire (pts (xy 125.73 85.725) (xy 128.27 85.725))
     (stroke (width 0) (type default) (color 0 0 0 0))
@@
     (stroke (width 0) (type default) (color 0 0 0 0))
   )
+  (wire (pts (xy 88.9 43.18) (xy 88.9 46.99))
+    (stroke (width 0) (type default) (color 0 0 0 0))
+  )
   (wire (pts (xy 32.385 90.17) (xy 36.83 90.17))
     (stroke (width 0) (type default) (color 0 0 0 0))
@@
     (stroke (width 0) (type default) (color 0 0 0 0))
   )
+  (wire (pts (xy 231.14 55.88) (xy 231.14 52.705))
+    (stroke (width 0) (type default) (color 0 0 0 0))
+  )
   (wire (pts (xy 172.466 241.427) (xy 190.246 241.427))
     (stroke (width 0) (type default) (color 0 0 0 0))
@@
     (stroke (width 0) (type default) (color 0 0 0 0))
   )
+  (wire (pts (xy 88.9 56.515) (xy 88.9 52.07))
+    (stroke (width 0) (type default) (color 0 0 0 0))
+  )
   (wire (pts (xy 348.615 320.04) (xy 344.17 320.04))
     (stroke (width 0) (type default) (color 0 0 0 0))
@@
     (stroke (width 0) (type default) (color 0 0 0 0))
   )
+  (wire (pts (xy 231.14 34.29) (xy 231.14 38.1))
+    (stroke (width 0) (type default) (color 0 0 0 0))
+  )
   (wire (pts (xy 88.392 244.475) (xy 85.852 244.475))
     (stroke (width 0) (type default) (color 0 0 0 0))
@@
     (pin "1")
   )
+  (symbol (lib_id "Device:LED_Small") (at 231.14 40.64 90) (unit 1)
+    (in_bom yes) (on_board yes)
+    (property "Reference" "D?" (id 0) (at 226.06 40.64 0))
+    (property "Value" "LED_Small" (id 1) (at 227.965 40.64 0))
+    (property "Footprint" "" (id 2) (at 231.14 40.64 90)
+      (effects (font (size 1.27 1.27)) hide)
+    )
+    (property "Datasheet" "~" (id 3) (at 231.14 40.64 90)
+      (effects (font (size 1.27 1.27)) hide)
+    )
+    (pin "1")
+    (pin "2")
+  )
+  (symbol (lib_id "power:GND") (at 231.14 55.88 0) (unit 1)
+    (in_bom yes) (on_board yes)
+    (property "Reference" "#PWR?" (id 0) (at 231.14 62.23 0)
+      (effects (font (size 1.27 1.27)) hide)
+    )
+    (property "Value" "GND" (id 1) (at 231.14 59.69 0))
+    (property "Footprint" "" (id 2) (at 231.14 55.88 0)
+      (effects (font (size 1.27 1.27)) hide)
+    )
+    (property "Datasheet" "" (id 3) (at 231.14 55.88 0)
+      (effects (font (size 1.27 1.27)) hide)
+    )
+    (pin "1")
+  )
   (symbol (lib_id "power:VCC") (at 103.632 231.775 0) (unit 1)
     (in_bom yes) (on_board yes) (fields_autoplaced)
@@
     (pin "2")
   )
+  (symbol (lib_id "Device:LED_Small") (at 88.9 49.53 90) (unit 1)
+    (in_bom yes) (on_board yes)
+    (property "Reference" "D?" (id 0) (at 83.82 49.53 0))
+    (property "Value" "LED_Small" (id 1) (at 85.725 49.53 0))
+    (property "Footprint" "" (id 2) (at 88.9 49.53 90)
+      (effects (font (size 1.27 1.27)) hide)
+    )
+    (property "Datasheet" "~" (id 3) (at 88.9 49.53 90)
+      (effects (font (size 1.27 1.27)) hide)
+    )
+    (pin "1")
+    (pin "2")
+  )
   (symbol (lib_id "power:+5V") (at 435.61 218.44 0) (unit 1)
     (in_bom yes) (on_board yes)
@@
     (pin "1")
   )
+  (symbol (lib_id "power:VBUS") (at 88.9 43.18 0) (unit 1)
+    (in_bom yes) (on_board yes) (fields_autoplaced)
+    (property "Reference" "#PWR?" (id 0) (at 88.9 46.99 0)
+      (effects (font (size 1.27 1.27)) hide)
+    )
+    (property "Value" "VBUS" (id 1) (at 88.9 38.1 0))
+    (property "Footprint" "" (id 2) (at 88.9 43.18 0)
+      (effects (font (size 1.27 1.27)) hide)
+    )
+    (property "Datasheet" "" (id 3) (at 88.9 43.18 0)
+      (effects (font (size 1.27 1.27)) hide)
+    )
+    (pin "1")
+  )
   (symbol (lib_id "Device:R_Small") (at 360.68 320.04 270) (mirror x) (unit 1)
     (in_bom yes) (on_board yes)
@@
     (pin "1")
   )
+  (symbol (lib_id "power:+5V") (at 231.14 34.29 0) (unit 1)
+    (in_bom yes) (on_board yes)
+    (property "Reference" "#PWR?" (id 0) (at 231.14 38.1 0)
+      (effects (font (size 1.27 1.27)) hide)
+    )
+    (property "Value" "+5V" (id 1) (at 231.14 30.48 0))
+    (property "Footprint" "" (id 2) (at 231.14 34.29 0)
+      (effects (font (size 1.27 1.27)) hide)
+    )
+    (property "Datasheet" "" (id 3) (at 231.14 34.29 0)
+      (effects (font (size 1.27 1.27)) hide)
+    )
+    (pin "1")
+  )
   (symbol (lib_id "LED:WS2812B") (at 369.57 120.015 0) (unit 1)
     (in_bom yes) (on_board yes)
@@
     (pin "2")
   )
+  (symbol (lib_id "Device:R_Small") (at 231.14 50.165 180) (unit 1)
+    (in_bom yes) (on_board yes)
+    (property "Reference" "R?" (id 0) (at 227.33 50.165 90))
+    (property "Value" "1k" (id 1) (at 229.235 50.165 90))
+    (property "Footprint" "Resistor_SMD:R_0805_2012Metric" (id 2) (at 231.14 50.165 0)
+      (effects (font (size 1.27 1.27)) hide)
+    )
+    (property "Datasheet" "~" (id 3) (at 231.14 50.165 0)
+      (effects (font (size 1.27 1.27)) hide)
+    )
+    (pin "1")
+    (pin "2")
+  )
   (symbol (lib_id "power:GND") (at 230.505 89.535 0) (unit 1)
     (in_bom yes) (on_board yes)
@@
     (pin "2")
   )
+  (symbol (lib_id "Device:R_Small") (at 88.9 59.055 180) (unit 1)
+    (in_bom yes) (on_board yes)
+    (property "Reference" "R?" (id 0) (at 85.09 59.055 90))
+    (property "Value" "1k" (id 1) (at 86.995 59.055 90))
+    (property "Footprint" "Resistor_SMD:R_0805_2012Metric" (id 2) (at 88.9 59.055 0)
+      (effects (font (size 1.27 1.27)) hide)
+    )
+    (property "Datasheet" "~" (id 3) (at 88.9 59.055 0)
+      (effects (font (size 1.27 1.27)) hide)
+    )
+    (pin "1")
+    (pin "2")
+  )
   (symbol (lib_id "LED:WS2812B") (at 402.59 41.91 0) (unit 1)
     (in_bom yes) (on_board yes)
@@
     (pin "1")
   )
+  (symbol (lib_id "power:GND") (at 88.9 64.77 0) (unit 1)
+    (in_bom yes) (on_board yes)
+    (property "Reference" "#PWR?" (id 0) (at 88.9 71.12 0)
+      (effects (font (size 1.27 1.27)) hide)
+    )
+    (property "Value" "GND" (id 1) (at 88.9 68.58 0))
+    (property "Footprint" "" (id 2) (at 88.9 64.77 0)
+      (effects (font (size 1.27 1.27)) hide)
+    )
+    (property "Datasheet" "" (id 3) (at 88.9 64.77 0)
+      (effects (font (size 1.27 1.27)) hide)
+    )
+    (pin "1")
+  )
   (symbol (lib_id "LED:WS2812B") (at 435.61 172.72 0) (unit 1)
     (in_bom yes) (on_board yes)
@@
       (reference "#PWR0251") (unit 1) (value "+5V") (footprint "")
     )
+    (path "/20eca63c-90e6-4032-aac9-6261fc70c0a9"
+      (reference "#PWR?") (unit 1) (value "GND") (footprint "")
+    )
+    (path "/48f48139-4e51-4209-a347-fa8cfba55fcf"
+      (reference "#PWR?") (unit 1) (value "VBUS") (footprint "")
+    )
+    (path "/6e3b3c43-d3f2-4580-aea2-55688637977e"
+      (reference "#PWR?") (unit 1) (value "+5V") (footprint "")
+    )
+    (path "/ea78ab63-06bb-43f6-9174-08b410d49290"
+      (reference "#PWR?") (unit 1) (value "GND") (footprint "")
+    )
     (path "/4d949544-83cc-4aec-998d-0bf78715ffa7"
       (reference "C1") (unit 1) (value "0-50pF") (footprint "Capacitor_SMD:C_0805_2012Metric")
@@
       (reference "D100") (unit 1) (value "LED_Small") (footprint "")
     )
+    (path "/20b8daa4-ecac-4d2a-b01b-15c85b2d75a6"
+      (reference "D?") (unit 1) (value "LED_Small") (footprint "")
+    )
+    (path "/39d654a4-49ec-4cdf-a738-a3c244be120b"
+      (reference "D?") (unit 1) (value "LED_Small") (footprint "")
+    )
     (path "/cda3a7e3-6804-4d5b-a507-5be364ac3196"
       (reference "J1") (unit 1) (value "TYPE-C-31-M-12") (footprint "Snapeda:TYPE-C-31-M-12_HRO_TYPE-C-31-M-12")
@@
       (reference "R8") (unit 1) (value "1k") (footprint "Resistor_SMD:R_0805_2012Metric")
     )
+    (path "/8652c87d-083c-4549-b2d7-e77581781219"
+      (reference "R?") (unit 1) (value "1k") (footprint "Resistor_SMD:R_0805_2012Metric")
+    )
+    (path "/976ea957-cbb1-4f0c-8875-c0921ecaefc2"
+      (reference "R?") (unit 1) (value "1k") (footprint "Resistor_SMD:R_0805_2012Metric")
+    )
     (path "/f4a5479e-f54a-497f-b04b-3b20cc56af37"

Commit message: update
Parts:
- C17: renamed from C20; footprint (none) -> Capacitor_SMD:C_0805_2012Metric
- C18: renamed from C22; footprint (none) -> Capacitor_SMD:C_0805_2012Metric
- C19: renamed from C24; footprint (none) -> Capacitor_SMD:C_0805_2012Metric
- C20: renamed from C9; footprint (none) -> Capacitor_SMD:C_0805_2012Metric
- C21: footprint (none) -> Capacitor_SMD:C_0805_2012Metric
- C22: renamed from C23; footprint (none) -> Capacitor_SMD:C_0805_2012Metric
- C23: renamed from C25; footprint (none) -> Capacitor_SMD:C_0805_2012Metric
- C24: renamed from C14; footprint (none) -> Capacitor_SMD:C_0805_2012Metric
- C25: renamed from C15; footprint (none) -> Capacitor_SMD:C_0805_2012Metric
- C26: value C_Small -> 0.1uF; footprint (none) -> Capacitor_SMD:C_0805_2012Metric
- C27: value C_Small -> 10uF; footprint (none) -> Capacitor_SMD:C_0805_2012Metric
- D100: renamed from D2; value LED_Small -> STAT; footprint (none) -> LED_SMD:LED_0603_1608Metric
- D101: renamed from D99; value LED_Small -> Red; footprint (none) -> LED_SMD:LED_0603_1608Metric
- D102: renamed from D100; value LED_Small -> Green; footprint (none) -> LED_SMD:LED_0603_1608Metric
- D97: renamed from D?; value LED_Small -> 5V; footprint (none) -> LED_SMD:LED_0603_1608Metric
- D98: renamed from D?; value LED_Small -> VBUS; footprint (none) -> LED_SMD:LED_0603_1608Metric
- D99: renamed from D1; value LED_Small -> INOKB; footprint (none) -> LED_SMD:LED_0603_1608Metric
- JP17: renamed from JP9; footprint (none) -> LED_SMD:LED_0603_1608Metric
- L1: footprint (none) -> Inductor_SMD:L_0805_2012Metric
- TP10, TP9: footprint (none) -> TestPoint:TestPoint_Pad_4.0x4.0mm
- U1: renamed from U3; footprint Package_TO_SOT_SMD:SOT-23-6_Handsoldering -> Package_TO_SOT_SMD:SOT-23-6
- U2: renamed from U4; footprint Package_TO_SOT_SMD:SOT-23-6_Handsoldering -> Package_TO_SOT_SMD:SOT-23-6
- U3: renamed from U1; footprint Package_TO_SOT_SMD:SOT-23-6_Handsoldering -> Package_TO_SOT_SMD:SOT-23-6
- U4: renamed from U2; footprint Package_TO_SOT_SMD:SOT-23-6_Handsoldering -> Package_TO_SOT_SMD:SOT-23-6
- U5: renamed from U8; footprint Package_TO_SOT_SMD:SOT-23-6_Handsoldering -> Package_TO_SOT_SMD:SOT-23-6
- U6: renamed from U9; footprint Package_TO_SOT_SMD:SOT-23-6_Handsoldering -> Package_TO_SOT_SMD:SOT-23-6
- U7: renamed from U6; footprint Package_TO_SOT_SMD:SOT-23-6_Handsoldering -> Package_TO_SOT_SMD:SOT-23-6
- U8: renamed from U7; footprint Package_TO_SOT_SMD:SOT-23-6_Handsoldering -> Package_TO_SOT_SMD:SOT-23-6
- gave numbers to parts that had none: 2
- renumbered C3 to C1, C13 to C10, C10 to C11, C11 to C12, C18 to C13, C19 to C14, C16 to C15, C17 to C16, C4 to C2, C1 to C3, C2 to C4, C8 to C5, C5 to C6, C6 to C8, C12 to C9, D3 to D1, D75 to D10, D83 to D11, D91 to D12, D4 to D13, D12 to D14, D20 to D15, D28 to D16, D36 to D17, D44 to D18, D52 to D19, D11 to D2, D60 to D20, D68 to D21, D76 to D22, D84 to D23, D92 to D24, D5 to D25, D13 to D26, D21 to D27, D29 to D28, D37 to D29, D19 to D3, D45 to D30, D53 to D31, D61 to D32, D69 to D33, D77 to D34, D85 to D35, D93 to D36, D6 to D37, D14 to D38, D22 to D39, D27 to D4, D30 to D40, D38 to D41, D46 to D42, D54 to D43, D62 to D44, D70 to D45, D78 to D46, D86 to D47, D94 to D48, D7 to D49, D35 to D5, D15 to D50, D23 to D51, D31 to D52, D39 to D53, D47 to D54, D63 to D56, D71 to D57, D79 to D58, D87 to D59, D43 to D6, D95 to D60, D8 to D61, D16 to D62, D24 to D63, D32 to D64, D40 to D65, D48 to D66, D56 to D67, D64 to D68, D72 to D69, D51 to D7, D80 to D70, D88 to D71, D96 to D72, D9 to D73, D17 to D74, D25 to D75, D33 to D76, D41 to D77, D49 to D78, D57 to D79, D59 to D8, D65 to D80, D73 to D81, D81 to D82, D89 to D83, D97 to D84, D10 to D85, D18 to D86, D26 to D87, D34 to D88, D42 to D89, D67 to D9, D50 to D90, D58 to D91, D66 to D92, D74 to D93, D82 to D94, D90 to D95, D98 to D96, JP5 to JP1, JP15 to JP10, JP16 to JP11, JP17 to JP12, JP10 to JP13, JP11 to JP14, JP12 to JP15, JP13 to JP16, JP6 to JP2, JP7 to JP3, JP8 to JP4, JP1 to JP5, JP2 to JP6, JP3 to JP7, JP4 to JP8, JP14 to JP9, R8 to R10, R5 to R3, R1 to R4, R6 to R5, R2 to R6, R3 to R7, R4 to R8, R7 to R9, TP4 to TP1, TP1 to TP2, TP2 to TP4, TP7 to TP5, TP8 to TP6, TP5 to TP7, TP6 to TP8, U5 to U9
Other:
- moved on the sheet: C11, C15, C16, C5, JP13, JP14, TP1, TP7, TP8, U7

Commit message: update
Parts:
- U9: footprint Snapeda:MAX77751CEFG_T_IC_MAX77751CEFG_T -> Snapeda:IC_MAX77751CEFG_T
Connections:
- net SYS is gone; now on net +5V: L1.2
- net BAT: now reaches C17.2, TP9.1, U9.13_14 (BATT)
Changed lines of the file:
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@@
     (stroke (width 0) (type default) (color 0 0 0 0))
   )
+  (wire (pts (xy 196.215 118.11) (xy 201.295 118.11))
+    (stroke (width 0) (type default) (color 0 0 0 0))
+  )
   (wire (pts (xy 64.135 278.765) (xy 67.945 278.765))
     (stroke (width 0) (type default) (color 0 0 0 0))
@@
     )
   )
-  (global_label "SYS" (shape input) (at 201.295 118.11 270) (fields_autoplaced)
-    (effects (font (size 1.27 1.27)) (justify right))
-    (property "Referenzen zwischen Schaltplänen" "${INTERSHEET_REFS}" (id 0) (at 201.3744 123.9418 90)
-      (effects (font (size 1.27 1.27)) (justify right) hide)
-    )
-  )
   (global_label "2out" (shape input) (at 558.8 67.945 0) (fields_autoplaced)
     (effects (font (size 1.27 1.27)) (justify left))
@@
     )
   )
+  (global_label "BAT" (shape input) (at 186.69 70.485 90) (fields_autoplaced)
+    (effects (font (size 1.27 1.27)) (justify left))
+    (property "Referenzen zwischen Schaltplänen" "${INTERSHEET_REFS}" (id 0) (at 186.6106 64.8346 90)
+      (effects (font (size 1.27 1.27)) (justify left) hide)
+    )
+  )
   (global_label "touch_point_8" (shape input) (at 400.685 332.74 0) (fields_autoplaced)
     (effects (font (size 1.27 1.27)) (justify left))
@@
     (property "Reference" "U9" (id 0) (at 161.925 62.23 0))
     (property "Value" "MAX77751CEFG_T" (id 1) (at 161.925 64.77 0))
-    (property "Footprint" "Snapeda:MAX77751CEFG_T_IC_MAX77751CEFG_T" (id 2) (at 161.925 90.805 0)
+    (property "Footprint" "Snapeda:IC_MAX77751CEFG_T" (id 2) (at 161.925 90.805 0)
       (effects (font (size 1.27 1.27)) (justify bottom) hide)
     )
@@
     (pin "4")
   )
+  (symbol (lib_id "power:+5V") (at 196.215 118.11 0) (unit 1)
+    (in_bom yes) (on_board yes)
+    (property "Reference" "#PWR?" (id 0) (at 196.215 121.92 0)
+      (effects (font (size 1.27 1.27)) hide)
+    )
+    (property "Value" "+5V" (id 1) (at 196.215 114.3 0))
+    (property "Footprint" "" (id 2) (at 196.215 118.11 0)
+      (effects (font (size 1.27 1.27)) hide)
+    )
+    (property "Datasheet" "" (id 3) (at 196.215 118.11 0)
+      (effects (font (size 1.27 1.27)) hide)
+    )
+    (pin "1")
+  )
   (symbol (lib_id "power:+5V") (at 340.995 320.04 0) (mirror y) (unit 1)
     (in_bom yes) (on_board yes)
@@
       (reference "#PWR0255") (unit 1) (value "GND") (footprint "")
     )
+    (path "/e1406b4f-a2c2-4e53-8d5b-e22f2d83d6a5"
+      (reference "#PWR?") (unit 1) (value "+5V") (footprint "")
+    )
     (path "/07d1a4e0-733f-4ad9-a5c8-74465e2c313d"
       (reference "C1") (unit 1) (value "0-50pF") (footprint "Capacitor_SMD:C_0805_2012Metric")
@@
     )
     (path "/615c5a86-c180-4f6a-8918-afa219ee2de2"
-      (reference "U9") (unit 1) (value "MAX77751CEFG_T") (footprint "Snapeda:MAX77751CEFG_T_IC_MAX77751CEFG_T")
+      (reference "U9") (unit 1) (value "MAX77751CEFG_T") (footprint "Snapeda:IC_MAX77751CEFG_T")
     )
     (path "/a71cdeed-1051-4d62-bd94-dca0a19008a3"
